Commit message: updates files to use right and left naming

File: pal_robotiq_85_gripper/pal_robotiq_85_description/robots/pal_robotiq_85_gripper.urdf.xacro (robot description, xacro)
@@ -2,5 +2,4 @@
 <robot name="robotiq_85_gripper" xmlns:xacro="http://ros.org/wiki/xacro">
     <xacro:include filename="$(find pal_robotiq_85_description)/urdf/robotiq_85_gripper.urdf.xacro" />
-    <xacro:include filename="$(find pal_robotiq_85_description)/urdf/robotiq_85_kinova_coupler.urdf.xacro" />
     <xacro:property name="pi" value="3.1415"/>
     <xacro:property name="prefix" value=""/>
@@ -9,5 +8,5 @@
         <parent link="base_link"/>
         <child link="${prefix}robotiq_coupler_link"/>
-        <origin xyz="0 0 -0.02754" rpy="0 0 0"/>
+        <origin xyz="0.0 0.0 0.0" rpy="0 0 0"/>
     </joint>
     <link name="${prefix}robotiq_coupler_link">
@@ -24,5 +23,5 @@
         <inertial>
             <mass value="0.1" />
-            <origin xyz="0.0 0.0 0.02754" />
+            <origin xyz="0.0 0.0 0.0" />
             <inertia ixx = "0.000001" ixy = "0.000000" ixz = "0.000000"
                      iyx = "0.000000" iyy = "0.000001" iyz = "0.000000"
@@ -31,5 +30,5 @@
     </link>
     <xacro:robotiq_85_gripper prefix="${prefix}" parent="${prefix}robotiq_coupler_link" >
-        <origin xyz="0 0 -0.0" rpy="0 ${pi/2} 0"/>
+        <origin xyz="0 0 -0.02754" rpy="0 ${pi/2} 0"/>
     </xacro:robotiq_85_gripper>
 </robot>

File: pal_robotiq_85_gripper/pal_robotiq_85_description/urdf/robotiq_85_gripper.transmission.xacro (robot description, xacro)
@@ -4,5 +4,5 @@
     <transmission name="${prefix}gripper_finger1_trans">
         <type>transmission_interface/SimpleTransmission</type>
-        <joint name="${prefix}gripper_finger1_joint">
+        <joint name="${prefix}gripper_finger_left_joint">
             <hardwareInterface>hardware_interface/PositionJointInterface</hardwareInterface>
             <hardwareInterface>hardware_interface/JointStateInterface</hardwareInterface>
@@ -17,11 +17,11 @@
             <!-- loading plugin: mimic joints works in gazebo now -->
         <plugin filename="libroboticsgroup_gazebo_mimic_joint_plugin.so" name="${prefix}mimic_robotiq_85_1">
-            <joint>${prefix}gripper_finger1_joint</joint>
-            <mimicJoint>${prefix}gripper_finger2_joint</mimicJoint>
+            <joint>${prefix}gripper_finger_left_joint</joint>
+            <mimicJoint>${prefix}gripper_finger_right_joint</mimicJoint>
             <!--multiplier>1.0</multiplier>
             <offset>0.0</offset-->
         </plugin>
         <plugin filename="libroboticsgroup_gazebo_mimic_joint_plugin.so" name="${prefix}mimic_robotiq_85_2">
-            <joint>${prefix}gripper_finger1_joint</joint>
+            <joint>${prefix}gripper_finger_left_joint</joint>
             <mimicJoint>${prefix}gripper_finger2_inner_knuckle_joint</mimicJoint>
             <!--multiplier>1.0</multiplier>
@@ -29,5 +29,5 @@
         </plugin>
         <plugin filename="libroboticsgroup_gazebo_mimic_joint_plugin.so" name="${prefix}mimic_robotiq_85_3">
-            <joint>${prefix}gripper_finger1_joint</joint>
+            <joint>${prefix}gripper_finger_left_joint</joint>
             <mimicJoint>${prefix}gripper_finger1_inner_knuckle_joint</mimicJoint>
             <!--multiplier>1.0</multiplier>
@@ -35,5 +35,5 @@
         </plugin>
         <plugin filename="libroboticsgroup_gazebo_mimic_joint_plugin.so" name="${prefix}mimic_robotiq_85_4">
-            <joint>${prefix}gripper_finger1_joint</joint>
+            <joint>${prefix}gripper_finger_left_joint</joint>
             <mimicJoint>${prefix}gripper_finger1_finger_tip_joint</mimicJoint>
             <multiplier>-1.0</multiplier>
@@ -41,5 +41,5 @@
         </plugin>
         <plugin filename="libroboticsgroup_gazebo_mimic_joint_plugin.so" name="${prefix}mimic_robotiq_85_5">
-            <joint>${prefix}gripper_finger1_joint</joint>
+            <joint>${prefix}gripper_finger_left_joint</joint>
             <mimicJoint>${prefix}gripper_finger2_finger_tip_joint</mimicJoint>
             <multiplier>-1.0</multiplier>

File: pal_robotiq_85_gripper/pal_robotiq_85_description/urdf/robotiq_85_gripper.urdf.xacro (robot description, xacro)
@@ -34,5 +34,5 @@
             <kd>1.0</kd>
         </gazebo>
-        <joint name="${prefix}gripper_finger1_joint" type="revolute">
+        <joint name="${prefix}gripper_finger_left_joint" type="revolute">
             <parent link="${prefix}gripper_base_link"/>
             <child link="${prefix}gripper_finger1_knuckle_link"/>
@@ -41,5 +41,5 @@
             <limit lower="0.0" upper="0.804" velocity="2.0" effort="1000"/>
         </joint>
-        <joint name="${prefix}gripper_finger2_joint" type="revolute">
+        <joint name="${prefix}gripper_finger_right_joint" type="revolute">
             <parent link="${prefix}gripper_base_link"/>
             <child link="${prefix}gripper_finger2_knuckle_link"/>
@@ -47,5 +47,5 @@
             <origin rpy="0.0 0.0 0.0" xyz="0.05490451627 -0.03060114443 0.0"/>
             <limit lower="-3.14" upper="3.14" velocity="100.0" effort="1000"/>
-            <mimic joint="${prefix}gripper_finger1_joint"/>
+            <mimic joint="${prefix}gripper_finger_left_joint"/>
         </joint>
         <link name="${prefix}gripper_finger1_knuckle_link">
@@ -169,5 +169,5 @@
             <origin xyz="0.06142 0.0127 0" rpy="${pi} 0.0 0.0" />
             <limit lower="-3.14" upper="3.14" velocity="100.0" effort="0.1"/>
-            <mimic joint="${prefix}gripper_finger1_joint" offset="0"/>
+            <mimic joint="${prefix}gripper_finger_left_joint" offset="0"/>
         </joint>
         <joint name="${prefix}gripper_finger2_inner_knuckle_joint" type="continuous">
@@ -177,5 +177,5 @@
             <origin xyz="0.06142 -0.0127 0" rpy="0 0 0"/>
             <limit lower="-3.14" upper="3.14" velocity="100.0" effort="0.1"/>
-            <mimic joint="${prefix}gripper_finger1_joint" offset="0"/>
+            <mimic joint="${prefix}gripper_finger_left_joint" offset="0"/>
         </joint>
         <link name="${prefix}gripper_finger1_inner_knuckle_link">
@@ -237,5 +237,5 @@
             <origin xyz="0.04303959807 -0.03759940821 0.0" rpy="0.0 0.0 0.0"/>
             <limit lower="-3.14" upper="3.14" velocity="100.0" effort="0.1"/>
-            <mimic joint="${prefix}gripper_finger1_joint" multiplier="-1"/>
+            <mimic joint="${prefix}gripper_finger_left_joint" multiplier="-1"/>
         </joint>
         <joint name="${prefix}gripper_finger2_finger_tip_joint" type="continuous">
@@ -245,5 +245,5 @@
             <origin rpy="0.0 0.0 0.0" xyz="0.04303959807 -0.03759940821  0.0"/>
             <limit lower="-3.14" upper="3.14" velocity="100.0" effort="0.1"/>
-            <mimic joint="${prefix}gripper_finger1_joint" multiplier="-1"/>
+            <mimic joint="${prefix}gripper_finger_left_joint" multiplier="-1"/>
         </joint>
         <link name="${prefix}gripper_finger1_finger_tip_link">

Commit message: Update URDF from ROS Industrial repo

File: pal_robotiq_85_gripper/pal_robotiq_85_description/robots/pal_robotiq_85_gripper.urdf.xacro (robot description, xacro)
@@ -3,20 +3,24 @@
     <xacro:include filename="$(find pal_robotiq_85_description)/urdf/robotiq_85_gripper.urdf.xacro" />
     <xacro:property name="pi" value="3.1415"/>
-    <xacro:property name="prefix" value=""/>
+    <xacro:property name="prefix" value="gripper_"/>
     <link name="base_link"/>
-    <joint name="${prefix}pal_robotiq_coupler_joint" type="fixed">
+    <joint name="${prefix}coupler_joint" type="fixed">
         <parent link="base_link"/>
-        <child link="${prefix}robotiq_coupler_link"/>
+        <child link="${prefix}coupler_link"/>
         <origin xyz="0.0 0.0 0.0" rpy="0 0 0"/>
     </joint>
-    <link name="${prefix}robotiq_coupler_link">
+    <link name="${prefix}coupler_link">
         <visual>
+            <origin xyz="0 0 0.013771" rpy="0 0 0" />
             <geometry>
-                <mesh filename="package://pal_robotiq_85_description/meshes/visual/pal_robotiq_coupling.stl"/>
+                <cylinder length="0.027542" radius="0.0375"/>
+                <!--mesh filename="package://pal_robotiq_85_description/meshes/visual/pal_robotiq_coupling.stl"/-->
             </geometry>
         </visual>
         <collision>
+            <origin xyz="0 0 0.013771" rpy="0 0 0" />
             <geometry>
-                <mesh filename="package://pal_robotiq_85_description/meshes/visual/pal_robotiq_coupling.stl"/>
+                <cylinder length="0.027542" radius="0.0375"/>
+                <!--mesh filename="package://pal_robotiq_85_description/meshes/visual/pal_robotiq_coupling.stl"/-->
             </geometry>
         </collision>
@@ -29,6 +33,6 @@
         </inertial>
     </link>
-    <xacro:robotiq_85_gripper prefix="${prefix}" parent="${prefix}robotiq_coupler_link" >
-        <origin xyz="0 0 -0.02754" rpy="0 ${pi/2} 0"/>
+    <xacro:robotiq_85_gripper prefix="${prefix}" parent="${prefix}coupler_link" >
+        <origin xyz="0 0 0.02754" rpy="0 0 0"/>
     </xacro:robotiq_85_gripper>
 </robot>

File: pal_robotiq_85_gripper/pal_robotiq_85_description/urdf/robotiq_85_gripper.transmission.xacro (robot description, xacro)
@@ -2,11 +2,11 @@
 <robot xmlns:xacro="http://ros.org/wiki/xacro">
   <xacro:macro name="robotiq_85_gripper_transmission" params="prefix">
-    <transmission name="${prefix}gripper_finger1_trans">
+    <transmission name="${prefix}gripper_finger_trans">
         <type>transmission_interface/SimpleTransmission</type>
-        <joint name="${prefix}gripper_finger_left_joint">
+        <joint name="${prefix}finger_joint">
             <hardwareInterface>hardware_interface/PositionJointInterface</hardwareInterface>
             <hardwareInterface>hardware_interface/JointStateInterface</hardwareInterface>
         </joint>
-        <actuator name="${prefix}gripper_finger1_motor">
+        <actuator name="${prefix}finger_motor">
             <mechanicalReduction>1</mechanicalReduction>
             <hardwareInterface>hardware_interface/PositionJointInterface</hardwareInterface>
@@ -14,37 +14,4 @@
         </actuator>
     </transmission>
-    <gazebo>
-            <!-- loading plugin: mimic joints works in gazebo now -->
-        <plugin filename="libroboticsgroup_gazebo_mimic_joint_plugin.so" name="${prefix}mimic_robotiq_85_1">
-            <joint>${prefix}gripper_finger_left_joint</joint>
-            <mimicJoint>${prefix}gripper_finger_right_joint</mimicJoint>
-            <!--multiplier>1.0</multiplier>
-            <offset>0.0</offset-->
-        </plugin>
-        <plugin filename="libroboticsgroup_gazebo_mimic_joint_plugin.so" name="${prefix}mimic_robotiq_85_2">
-            <joint>${prefix}gripper_finger_left_joint</joint>
-            <mimicJoint>${prefix}gripper_finger2_inner_knuckle_joint</mimicJoint>
-            <!--multiplier>1.0</multiplier>
-            <offset>0.0</offset-->
-        </plugin>
-        <plugin filename="libroboticsgroup_gazebo_mimic_joint_plugin.so" name="${prefix}mimic_robotiq_85_3">
-            <joint>${prefix}gripper_finger_left_joint</joint>
-            <mimicJoint>${prefix}gripper_finger1_inner_knuckle_joint</mimicJoint>
-            <!--multiplier>1.0</multiplier>
-            <offset>0.0</offset-->
-        </plugin>
-        <plugin filename="libroboticsgroup_gazebo_mimic_joint_plugin.so" name="${prefix}mimic_robotiq_85_4">
-            <joint>${prefix}gripper_finger_left_joint</joint>
-            <mimicJoint>${prefix}gripper_finger1_finger_tip_joint</mimicJoint>
-            <multiplier>-1.0</multiplier>
-            <offset>0.0</offset>
-        </plugin>
-        <plugin filename="libroboticsgroup_gazebo_mimic_joint_plugin.so" name="${prefix}mimic_robotiq_85_5">
-            <joint>${prefix}gripper_finger_left_joint</joint>
-            <mimicJoint>${prefix}gripper_finger2_finger_tip_joint</mimicJoint>
-            <multiplier>-1.0</multiplier>
-            <offset>0.0</offset>
-        </plugin>
-    </gazebo>
   </xacro:macro>
 </robot>
