Commit message: Update URDF from ROS Industrial repo

File: pal_robotiq_85_gripper/pal_robotiq_85_description/urdf/robotiq_85_gripper.urdf.xacro (robot description, xacro)
@@ -1,303 +1,299 @@
 <?xml version="1.0"?>
-<robot name="robotiq_85_gripper" xmlns:xacro="http://ros.org/wiki/xacro">
-    <xacro:include filename="$(find pal_robotiq_85_description)/urdf/robotiq_85_gripper.transmission.xacro" />
-    <xacro:macro name="robotiq_85_gripper" params="prefix parent *origin">
-        <joint name="${prefix}gripper_base_joint" type="fixed">
-            <parent link="${parent}"/>
-            <child link="${prefix}gripper_base_link"/>
-            <xacro:insert_block name="origin"/>
-        </joint>
-        <link name="${prefix}gripper_base_link">
-            <visual>
-                <geometry>
-                    <mesh filename="package://pal_robotiq_85_description/meshes/visual/robotiq_85_base_link.stl"/>
-                </geometry>
-            </visual>
-            <collision>
-                <geometry>
-                    <mesh filename="package://pal_robotiq_85_description/meshes/collision/robotiq_85_base_link.dae"/>
-                </geometry>
-            </collision>
-            <inertial>
-                <mass value="0.636951" />
-                <origin xyz="0.0 0.0 0.0" />
-                <inertia ixx = "0.000380" ixy = "0.000000" ixz = "0.000000"
-                         iyx = "0.000000" iyy = "0.001110" iyz = "0.000000"
-                         izx = "0.000000" izy = "0.000000" izz = "0.001171" />
-            </inertial>
-        </link>
-        <gazebo reference="${prefix}gripper_base_link">
-            <implicitSpringDamper>1</implicitSpringDamper>
-            <mu1>100000</mu1>
-            <mu2>100000</mu2>
-            <kp>100000000.0</kp>
-            <kd>1.0</kd>
-        </gazebo>
-        <joint name="${prefix}gripper_finger_left_joint" type="revolute">
-            <parent link="${prefix}gripper_base_link"/>
-            <child link="${prefix}gripper_finger1_knuckle_link"/>
-            <axis xyz="0 0 1"/>
-            <origin rpy="${pi} 0.0 0.0" xyz="0.05490451627 0.03060114443 0.0"/>
-            <limit lower="0.0" upper="0.804" velocity="2.0" effort="1000"/>
-        </joint>
-        <joint name="${prefix}gripper_finger_right_joint" type="revolute">
-            <parent link="${prefix}gripper_base_link"/>
-            <child link="${prefix}gripper_finger2_knuckle_link"/>
-            <axis xyz="0 0 1"/>
-            <origin rpy="0.0 0.0 0.0" xyz="0.05490451627 -0.03060114443 0.0"/>
-            <limit lower="-3.14" upper="3.14" velocity="100.0" effort="1000"/>
-            <mimic joint="${prefix}gripper_finger_left_joint"/>
-        </joint>
-        <link name="${prefix}gripper_finger1_knuckle_link">
-            <visual>
-                <geometry>
-                    <mesh filename="package://pal_robotiq_85_description/meshes/visual/robotiq_85_knuckle_link.stl"/>
-                </geometry>
-            </visual>
-            <collision>
-                <geometry>
-                    <mesh filename="package://pal_robotiq_85_description/meshes/collision/robotiq_85_knuckle_link.dae"/>
-                </geometry>
-            </collision>
-            <inertial>
-                <mass value="0.018491" />
-                <origin xyz="0.0 0.0 0.0" />
-                <inertia ixx = "0.000009" ixy = "-0.000001" ixz = "0.000000"
-                         iyx = "-0.000001" iyy = "0.000001" iyz = "0.000000"
-                         izx = "0.000000" izy = "0.000000" izz = "0.000010" />
-            </inertial>
-        </link>
-        <gazebo reference="${prefix}gripper_finger1_knuckle_link">
-            <implicitSpringDamper>1</implicitSpringDamper>
-            <mu1>100000</mu1>
-            <mu2>100000</mu2>
-            <kp>100000000.0</kp>
-            <kd>1.0</kd>
-        </gazebo>
-        <link name="${prefix}gripper_finger2_knuckle_link">
-            <visual>
-                <geometry>
-                    <mesh filename="package://pal_robotiq_85_description/meshes/visual/robotiq_85_knuckle_link.stl"/>
-                </geometry>
-            </visual>
-            <collision>
-                <geometry>
-                    <mesh filename="package://pal_robotiq_85_description/meshes/collision/robotiq_85_knuckle_link.dae"/>
-                </geometry>
-            </collision>
-            <inertial>
-                <mass value="0.018491" />
-                <origin xyz="0.0 0.0 0.0" />
-                <inertia ixx = "0.000009" ixy = "-0.000001" ixz = "0.000000"
-                         iyx = "-0.000001" iyy = "0.000001" iyz = "0.000000"
-                         izx = "0.000000" izy = "0.000000" izz = "0.000010" />
-            </inertial>
-        </link>
-        <gazebo reference="${prefix}gripper_finger2_knuckle_link">
-            <implicitSpringDamper>1</implicitSpringDamper>
-            <mu1>100000</mu1>
-            <mu2>100000</mu2>
-            <kp>100000000.0</kp>
-            <kd>1.0</kd>
-        </gazebo>
-        <joint name="${prefix}gripper_finger1_finger_joint" type="fixed">
-            <parent link="${prefix}gripper_finger1_knuckle_link"/>
-            <child link="${prefix}gripper_finger1_finger_link"/>
-            <origin xyz="-0.00408552455 -0.03148604435 0.0" rpy="0 0 0" />
-        </joint>
-        <joint name="${prefix}gripper_finger2_finger_joint" type="fixed">
-            <parent link="${prefix}gripper_finger2_knuckle_link"/>
-            <child link="${prefix}gripper_finger2_finger_link"/>
-            <origin xyz="-0.00408552455 -0.03148604435 0.0" rpy="0 0 0" />
-        </joint>
-        <link name="${prefix}gripper_finger1_finger_link">
-            <visual>
-                <geometry>
-                    <mesh filename="package://pal_robotiq_85_description/meshes/visual/robotiq_85_finger_link.stl"/>
-                </geometry>
-            </visual>
-            <collision>
-                <geometry>
-                    <mesh filename="package://pal_robotiq_85_description/meshes/collision/robotiq_85_finger_link.dae"/>
-                </geometry>
-            </collision>
-            <inertial>
-                <mass value="0.027309" />
-                <origin xyz="0.0 0.0 0.0" />
-                <inertia ixx = "0.000003" ixy = "-0.000002" ixz = "0.000000"
-                         iyx = "-0.000002" iyy = "0.000021" iyz = "0.000000"
-                         izx = "0.000000" izy = "0.000000" izz = "0.000020" />
-            </inertial>
-        </link>
-        <gazebo reference="${prefix}gripper_finger1_finger_link">
-            <implicitSpringDamper>1</implicitSpringDamper>
-            <mu1>100000</mu1>
-            <mu2>100000</mu2>
-            <kp>100000000.0</kp>
-            <kd>1.0</kd>
-        </gazebo>
-        <link name="${prefix}gripper_finger2_finger_link">
-            <visual>
-                <geometry>
-                    <mesh filename="package://pal_robotiq_85_description/meshes/visual/robotiq_85_finger_link.stl"/>
-                </geometry>
-            </visual>
-            <collision>
-                <geometry>
-                    <mesh filename="package://pal_robotiq_85_description/meshes/collision/robotiq_85_finger_link.dae"/>
-                </geometry>
-            </collision>
-            <inertial>
-                <mass value="0.027309" />
-                <origin xyz="0.0 0.0 0.0" />
-                <inertia ixx = "0.000003" ixy = "-0.000002" ixz = "0.000000"
-                         iyx = "-0.000002" iyy = "0.000021" iyz = "0.000000"
-                         izx = "0.000000" izy = "0.000000" izz = "0.000020" />
-            </inertial>
-        </link>
-        <gazebo reference="${prefix}gripper_finger2_finger_link">
-            <implicitSpringDamper>1</implicitSpringDamper>
-            <mu1>100000</mu1>
-            <mu2>100000</mu2>
-            <kp>100000000.0</kp>
-            <kd>1.0</kd>
-        </gazebo>
-        <joint name="${prefix}gripper_finger1_inner_knuckle_joint" type="continuous">
-            <parent link="${prefix}gripper_base_link"/>
-            <child link="${prefix}gripper_finger1_inner_knuckle_link"/>
-            <axis xyz="0 0 1"/>
-            <origin xyz="0.06142 0.0127 0" rpy="${pi} 0.0 0.0" />
-            <limit lower="-3.14" upper="3.14" velocity="100.0" effort="0.1"/>
-            <mimic joint="${prefix}gripper_finger_left_joint" offset="0"/>
-        </joint>
-        <joint name="${prefix}gripper_finger2_inner_knuckle_joint" type="continuous">
-            <parent link="${prefix}gripper_base_link"/>
-            <child link="${prefix}gripper_finger2_inner_knuckle_link"/>
-            <axis xyz="0 0 1"/>
-            <origin xyz="0.06142 -0.0127 0" rpy="0 0 0"/>
-            <limit lower="-3.14" upper="3.14" velocity="100.0" effort="0.1"/>
-            <mimic joint="${prefix}gripper_finger_left_joint" offset="0"/>
-        </joint>
-        <link name="${prefix}gripper_finger1_inner_knuckle_link">
-            <visual>
-                <geometry>
-                    <mesh filename="package://pal_robotiq_85_description/meshes/visual/robotiq_85_inner_knuckle_link.stl"/>
-                </geometry>
-            </visual>
-            <collision>
-                <geometry>
-                    <mesh filename="package://pal_robotiq_85_description/meshes/collision/robotiq_85_inner_knuckle_link.dae"/>
-                </geometry>
-            </collision>
-            <inertial>
-                <mass value="0.029951" />
-                <origin xyz="0.0 0.0 0.0" />
-                <inertia ixx = "0.000039" ixy = "0.000000" ixz = "0.000000"
-                         iyx = "0.000000" iyy = "0.000005" iyz = "0.000000"
-                         izx = "0.000000" izy = "0.000000" izz = "0.000035" />
-            </inertial>
-        </link>
-        <gazebo reference="${prefix}gripper_finger1_inner_knuckle_link">
-            <implicitSpringDamper>1</implicitSpringDamper>
-            <mu1>100000</mu1>
-            <mu2>100000</mu2>
-            <kp>100000000.0</kp>
-            <kd>1.0</kd>
-        </gazebo>
-        <link name="${prefix}gripper_finger2_inner_knuckle_link">
-            <visual>
-                <geometry>
-                    <mesh filename="package://pal_robotiq_85_description/meshes/visual/robotiq_85_inner_knuckle_link.stl"/>
-                </geometry>
-            </visual>
-            <collision>
-                <geometry>
-                    <mesh filename="package://pal_robotiq_85_description/meshes/collision/robotiq_85_inner_knuckle_link.dae"/>
-                </geometry>
-            </collision>
-            <inertial>
-                <mass value="0.029951" />
-                <origin xyz="0.0 0.0 0.0" />
-                <inertia ixx = "0.000039" ixy = "0.000000" ixz = "0.000000"
-                         iyx = "0.000000" iyy = "0.000005" iyz = "0.000000"
-                         izx = "0.000000" izy = "0.000000" izz = "0.000035" />
-            </inertial>
-        </link>
-        <gazebo reference="${prefix}gripper_finger2_inner_knuckle_link">
-            <implicitSpringDamper>1</implicitSpringDamper>
-            <mu1>100000</mu1>
-            <mu2>100000</mu2>
-            <kp>100000000.0</kp>
-            <kd>1.0</kd>
-        </gazebo>
-        <joint name="${prefix}gripper_finger1_finger_tip_joint" type="continuous">
-            <parent link="${prefix}gripper_finger1_inner_knuckle_link"/>
-            <child link="${prefix}gripper_finger1_finger_tip_link"/>
-            <axis xyz="0 0 1"/>
-            <origin xyz="0.04303959807 -0.03759940821 0.0" rpy="0.0 0.0 0.0"/>
-            <limit lower="-3.14" upper="3.14" velocity="100.0" effort="0.1"/>
-            <mimic joint="${prefix}gripper_finger_left_joint" multiplier="-1"/>
-        </joint>
-        <joint name="${prefix}gripper_finger2_finger_tip_joint" type="continuous">
-            <parent link="${prefix}gripper_finger2_inner_knuckle_link"/>
-            <child link="${prefix}gripper_finger2_finger_tip_link"/>
-            <axis xyz="0 0 1"/>
-            <origin rpy="0.0 0.0 0.0" xyz="0.04303959807 -0.03759940821  0.0"/>
-            <limit lower="-3.14" upper="3.14" velocity="100.0" effort="0.1"/>
-            <mimic joint="${prefix}gripper_finger_left_joint" multiplier="-1"/>
-        </joint>
-        <link name="${prefix}gripper_finger1_finger_tip_link">
-            <visual>
-                <geometry>
-                    <mesh filename="package://pal_robotiq_85_description/meshes/visual/robotiq_85_finger_tip_link.stl"/>
-                </geometry>
-            </visual>
-            <collision>
-                <geometry>
-                    <mesh filename="package://pal_robotiq_85_description/meshes/collision/robotiq_85_finger_tip_link.dae"/>
-                </geometry>
-            </collision>
-            <inertial>
-                <mass value="0.019555" />
-                <origin xyz="0.0 0.0 0.0" />
-                <inertia ixx = "0.000002" ixy = "0.000000" ixz = "0.000000"
-                         iyx = "0.000000" iyy = "0.000005" iyz = "0.000000"
-                         izx = "0.000000" izy = "0.000000" izz = "0.000006" />
-            </inertial>
-        </link>
-        <gazebo reference="${prefix}gripper_finger1_finger_tip_link">
-            <implicitSpringDamper>1</implicitSpringDamper>
-            <mu1>100000</mu1>
-            <mu2>100000</mu2>
-            <kp>100000000.0</kp>
-            <kd>1.0</kd>
-        </gazebo>
-        <link name="${prefix}gripper_finger2_finger_tip_link">
-            <visual>
-                <geometry>
-                    <mesh filename="package://pal_robotiq_85_description/meshes/visual/robotiq_85_finger_tip_link.stl"/>
-                </geometry>
-            </visual>
-            <collision>
-                <geometry>
-                    <mesh filename="package://pal_robotiq_85_description/meshes/collision/robotiq_85_finger_tip_link.dae"/>
-                </geometry>
-            </collision>
-            <inertial>
-                <mass value="0.019555" />
-                <origin xyz="0.0 0.0 0.0" />
-                <inertia ixx = "0.000002" ixy = "0.000000" ixz = "0.000000"
-                         iyx = "0.000000" iyy = "0.000005" iyz = "0.000000"
-                         izx = "0.000000" izy = "0.000000" izz = "0.000006" />
-            </inertial>
-        </link>
-        <gazebo reference="${prefix}gripper_finger2_finger_tip_link">
-            <implicitSpringDamper>1</implicitSpringDamper>
-            <mu1>100000</mu1>
-            <mu2>100000</mu2>
-            <kp>100000000.0</kp>
-            <kd>1.0</kd>
-        </gazebo>
-        <xacro:robotiq_85_gripper_transmission prefix="${prefix}" />
-    </xacro:macro>
+<robot xmlns:xacro="http://ros.org/wiki/xacro">
+  <xacro:include filename="$(find pal_robotiq_85_description)/urdf/robotiq_85_gripper.transmission.xacro" />
+  <xacro:macro name="outer_knuckle" params="prefix fingerprefix ">
+    <link name="${prefix}${fingerprefix}_outer_knuckle">
+      <inertial>
+        <origin xyz="-0.000200000000003065 0.0199435877845359 0.0292245259211331" rpy="0 0 0" />
+        <mass value="0.00853198276973456" />
+        <inertia ixx="2.89328108496468E-06" ixy="-1.57935047237397E-19" ixz="-1.93980378593255E-19" iyy="1.86719750325683E-06" iyz="-1.21858577871576E-06" izz="1.21905238907251E-06" />
+      </inertial>
+      <visual>
+        <origin xyz="0 0 0" rpy="0 0 0" />
+        <geometry>
+          <mesh filename="package://pal_robotiq_85_description/meshes/visual/robotiq_85_outer_knuckle.dae" scale="0.001 0.001 0.001"/>
+        </geometry>
+        <material name="">
+          <color rgba="0.792156862745098 0.819607843137255 0.933333333333333 1" />
+        </material>
+      </visual>
+      <collision>
+        <origin xyz="0 0 0" rpy="0 0 0" />
+        <geometry>
+          <mesh filename="package://pal_robotiq_85_description/meshes/collision/robotiq_85_outer_knuckle.dae" scale="0.001 0.001 0.001"/>
+        </geometry>
+      </collision>
+    </link>
+    <gazebo reference="${prefix}${fingerprefix}_outer_knuckle">
+        <implicitSpringDamper>1</implicitSpringDamper>
+        <mu1>100000</mu1>
+        <mu2>100000</mu2>
+        <kp>100000000.0</kp>
+        <kd>1.0</kd>
+    </gazebo>
+  </xacro:macro>
+  <xacro:macro name="outer_finger" params="prefix fingerprefix ">
+    <link name="${prefix}${fingerprefix}_outer_finger">
+      <inertial>
+        <origin xyz="0.00030115855001899 0.0373907951953854 -0.0208027427000385" rpy="0 0 0" />
+        <mass value="0.022614240507152" />
+        <inertia ixx="1.52518312458174E-05" ixy="9.76583423954399E-10" ixz="-5.43838577022588E-10" iyy="6.17694243867776E-06" iyz="6.78636130740228E-06" izz="1.16494917907219E-05" />
+      </inertial>
+      <visual>
+        <origin xyz="0 0 0" rpy="0 0 0" />
+        <geometry>
+          <mesh filename="package://pal_robotiq_85_description/meshes/visual/robotiq_85_outer_finger.dae" scale="0.001 0.001 0.001"/>
+        </geometry>
+        <material name="">
+          <color rgba="0.1 0.1 0.1 1" />
+        </material>
+      </visual>
+      <collision>
+        <origin xyz="0 0 0" rpy="0 0 0" />
+        <geometry>
+          <mesh filename="package://pal_robotiq_85_description/meshes/collision/robotiq_85_outer_finger.dae" scale="0.001 0.001 0.001"/>
+        </geometry>
+      </collision>
+    </link>
+    <gazebo reference="{prefix}${fingerprefix}_outer_finger">
+        <implicitSpringDamper>1</implicitSpringDamper>
+        <mu1>100000</mu1>
+        <mu2>100000</mu2>
+        <kp>100000000.0</kp>
+        <kd>1.0</kd>
+    </gazebo>
+  </xacro:macro>
+  <xacro:macro name="inner_knuckle" params="prefix fingerprefix ">
+    <link name="${prefix}${fingerprefix}_inner_knuckle">
+      <inertial>
+        <origin xyz="0.000123011831763771 0.0507850843201817 0.00103968640075166" rpy="0 0 0" />
+       <mass value="0.0271177346495152" />
+        <inertia ixx="2.61910379223783E-05" ixy="-2.43616858946494E-07" ixz="-6.37789906117123E-09" iyy="2.8270243746167E-06" iyz="-5.37200748039765E-07" izz="2.83695868220296E-05" />
+      </inertial>
+      <visual>
+        <origin xyz="0 0 0" rpy="0 0 0" />
+        <geometry>
+          <mesh filename="package://pal_robotiq_85_description/meshes/visual/robotiq_85_inner_knuckle.dae" scale="0.001 0.001 0.001"/>
+        </geometry>
+        <material name="">
+          <color rgba="0.1 0.1 0.1 1" />
+        </material>
+      </visual>
+      <collision>
+        <origin xyz="0 0 0" rpy="0 0 0" />
+        <geometry>
+          <mesh filename="package://pal_robotiq_85_description/meshes/collision/robotiq_85_inner_knuckle.dae" scale="0.001 0.001 0.001"/>
+        </geometry>
+      </collision>
+    </link>
+    <gazebo reference="${prefix}${fingerprefix}_inner_knuckle">
+        <implicitSpringDamper>1</implicitSpringDamper>
+        <mu1>100000</mu1>
+        <mu2>100000</mu2>
+        <kp>100000000.0</kp>
+        <kd>1.0</kd>
+    </gazebo>
+  </xacro:macro>
+  <xacro:macro name="inner_finger" params="prefix fingerprefix ">
+    <link name="${prefix}${fingerprefix}_inner_finger">
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