Commit message: Move the coupling link into the macro and update links

File: pal_robotiq_85_gripper/pal_robotiq_85_description/robots/pal_robotiq_85_gripper.urdf.xacro (robot description, xacro)
@@ -5,34 +5,6 @@
     <xacro:property name="prefix" value="gripper_"/>
     <link name="base_link"/>
-    <joint name="${prefix}coupler_joint" type="fixed">
-        <parent link="base_link"/>
-        <child link="${prefix}coupler_link"/>
-        <origin xyz="0.0 0.0 0.0" rpy="0 0 0"/>
-    </joint>
-    <link name="${prefix}coupler_link">
-        <visual>
-            <origin xyz="0 0 0.013771" rpy="0 0 0" />
-            <geometry>
-                <cylinder length="0.027542" radius="0.0375"/>
-                <!--mesh filename="package://pal_robotiq_85_description/meshes/visual/pal_robotiq_coupling.stl"/-->
-            </geometry>
-        </visual>
-        <collision>
-            <origin xyz="0 0 0.013771" rpy="0 0 0" />
-            <geometry>
-                <cylinder length="0.027542" radius="0.0375"/>
-                <!--mesh filename="package://pal_robotiq_85_description/meshes/visual/pal_robotiq_coupling.stl"/-->
-            </geometry>
-        </collision>
-        <inertial>
-            <mass value="0.1" />
-            <origin xyz="0.0 0.0 0.0" />
-            <inertia ixx = "0.000001" ixy = "0.000000" ixz = "0.000000"
-                     iyx = "0.000000" iyy = "0.000001" iyz = "0.000000"
-                     izx = "0.000000" izy = "0.000000" izz = "0.000001" />
-        </inertial>
-    </link>
-    <xacro:robotiq_85_gripper prefix="${prefix}" parent="${prefix}coupler_link" >
-        <origin xyz="0 0 0.02754" rpy="0 0 0"/>
+    <xacro:robotiq_85_gripper prefix="${prefix}" parent="base_link" >
+        <origin xyz="0 0 0" rpy="0 0 0"/>
     </xacro:robotiq_85_gripper>
 </robot>

File: pal_robotiq_85_gripper/pal_robotiq_85_description/urdf/robotiq_85_gripper.urdf.xacro (robot description, xacro)
@@ -235,9 +235,41 @@
     </link>
   </xacro:macro>
-  <xacro:macro name="robotiq_base_joint" params="prefix parent *origin">
-    <joint name="${prefix}gripper_base_joint" type="fixed">
+  <xacro:macro name="pal_robotiq_coupling_link" params="prefix">
+    <link name="${prefix}coupler_link">
+        <visual>
+            <origin xyz="0 0 0.013771" rpy="0 0 0" />
+            <geometry>
+                <cylinder length="0.027542" radius="0.0375"/>
+                <!--mesh filename="package://pal_robotiq_85_description/meshes/visual/pal_robotiq_coupling.stl"/-->
+            </geometry>
+        </visual>
+        <collision>
+            <origin xyz="0 0 0.013771" rpy="0 0 0" />
+            <geometry>
+                <cylinder length="0.027542" radius="0.0375"/>
+                <!--mesh filename="package://pal_robotiq_85_description/meshes/visual/pal_robotiq_coupling.stl"/-->
+            </geometry>
+        </collision>
+        <inertial>
+            <mass value="0.1" />
+            <origin xyz="0.0 0.0 0.0" />
+            <inertia ixx = "0.000001" ixy = "0.000000" ixz = "0.000000"
+                     iyx = "0.000000" iyy = "0.000001" iyz = "0.000000"
+                     izx = "0.000000" izy = "0.000000" izz = "0.000001" />
+        </inertial>
+    </link>
+  </xacro:macro>
+  <xacro:macro name="pal_robotiq_coupling_joint" params="prefix parent *origin">
+    <joint name="${prefix}coupler_joint" type="fixed">
       <parent link="${parent}"/>
+      <child link="${prefix}coupler_link"/>
+      <xacro:insert_block name="origin"/>
+    </joint>
+  </xacro:macro>
+  <xacro:macro name="robotiq_base_joint" params="prefix">
+    <joint name="${prefix}base_joint" type="fixed">
+      <parent link="${prefix}coupler_link"/>
       <child link="${prefix}base_link"/>
-      <xacro:insert_block name="origin"/>
+      <origin xyz="0 0 0.02754" rpy="0 0 0"/>
     </joint>
   </xacro:macro>
@@ -288,9 +320,11 @@
   <xacro:macro name="robotiq_85_gripper" params="prefix parent *origin">
     <xacro:robotiq_base_link prefix="${prefix}"/>
+    <xacro:pal_robotiq_coupling_link prefix="${prefix}"/>
     <xacro:finger_links prefix="${prefix}" fingerprefix="left" />
     <xacro:finger_links prefix="${prefix}" fingerprefix="right"/>
-    <xacro:robotiq_base_joint prefix="${prefix}" parent="${parent}">
+    <xacro:robotiq_base_joint prefix="${prefix}" />
+    <xacro:pal_robotiq_coupling_joint prefix="${prefix}" parent="${parent}">
       <xacro:insert_block name="origin" />
-    </xacro:robotiq_base_joint>
+    </xacro:pal_robotiq_coupling_joint>
     <xacro:finger_joint prefix="${prefix}"/>
     <xacro:right_outer_knuckle_joint prefix="${prefix}"/>

Commit message: Update URDF of robotiq 85

File: pal_robotiq_85_gripper/pal_robotiq_85_description/robots/pal_robotiq_85_gripper.urdf.xacro (robot description, xacro)
@@ -4,7 +4,38 @@
     <xacro:property name="pi" value="3.1415"/>
     <xacro:property name="prefix" value="gripper_"/>
-    <link name="base_link"/>
-    <xacro:robotiq_85_gripper prefix="${prefix}" parent="base_link" >
+    <gazebo>
+        <plugin name="gazebo_ros_control" filename="libgazebo_ros_control.so">
+            <robotNamespace></robotNamespace>
+        </plugin>
+    </gazebo>
+    <link name="world"/>
+    <joint name="world_fixed" type="fixed">
         <origin xyz="0 0 0" rpy="0 0 0"/>
+        <parent link="world"/>
+        <child link="gripper_root_link"/>
+    </joint>
+    <link name="gripper_root_link">
+        <visual>
+            <origin xyz="0 0 0.5" rpy="0 0 0"/>
+            <geometry>
+                <box size="0.1 0.1 1.0"/>
+            </geometry>
+        </visual>
+        <collision>
+            <origin xyz="0 0 0.5" rpy="0 0 0"/>
+            <geometry>
+                <box size="0.1 0.1 1.0"/>
+            </geometry>
+        </collision>
+        <inertial>
+            <mass value="1e2" />
+            <origin xyz="0.0 0.0 0.0" />
+            <inertia ixx = "0.000001" ixy = "0.000000" ixz = "0.000000"
+                     iyx = "0.000000" iyy = "0.000001" iyz = "0.000000"
+                     izx = "0.000000" izy = "0.000000" izz = "0.000001" />
+        </inertial>
+    </link>
+    <xacro:robotiq_85_gripper prefix="${prefix}" parent="gripper_root_link" >
+        <origin xyz="0.05 0 0.85" rpy="0 1.5708 0"/>
     </xacro:robotiq_85_gripper>
 </robot>

File: pal_robotiq_85_gripper/pal_robotiq_85_description/urdf/robotiq_85_gripper.urdf.xacro (robot description, xacro)
@@ -236,21 +236,19 @@
   </xacro:macro>
   <xacro:macro name="pal_robotiq_coupling_link" params="prefix">
-    <material name="black">
-      <color rgba="0 0 0 1"/>
-    </material>
     <link name="${prefix}coupler_link">
+      <material name="black">
+        <color rgba="0 0 0 1"/>
+      </material>
         <visual>
-            <origin xyz="0 0 0.013771" rpy="0 0 0" />
+            <origin xyz="0 0 0.0" rpy="3.1416 0 0" />
             <geometry>
-                <cylinder length="0.027542" radius="0.0375"/>
-                <!--mesh filename="package://pal_robotiq_85_description/meshes/visual/pal_robotiq_coupling.stl"/-->
+                <mesh filename="package://pal_robotiq_85_description/meshes/visual/pal_robotiq_coupling.stl"/>
             </geometry>
             <material name="black"/>
         </visual>
         <collision>
-            <origin xyz="0 0 0.013771" rpy="0 0 0" />
+            <origin xyz="0 0 0.0" rpy="3.1416 0 0" />
             <geometry>
-                <cylinder length="0.027542" radius="0.0375"/>
-                <!--mesh filename="package://pal_robotiq_85_description/meshes/visual/pal_robotiq_coupling.stl"/-->
+                <mesh filename="package://pal_robotiq_85_description/meshes/visual/pal_robotiq_coupling.stl"/>
             </geometry>
         </collision>
