Commit message: Add config files for epick gripper

File: pal_robotiq_epick_gripper/pal_robotiq_epick_description/robots/pal_robotiq_epick_gripper.urdf.xacro (robot description, xacro)
@@ -1,4 +1,5 @@
 <?xml version="1.0" ?>
 <robot name="robotiq_epick_gripper" xmlns:xacro="http://ros.org/wiki/xacro">
+    <xacro:include filename="$(find pal_robotiq_epick_description)/urdf/robotiq_epcick_gripper.transmission.xacro" />
     <xacro:include filename="$(find pal_robotiq_epick_description)/urdf/robotiq_epick_model_macro.xacro" />
     <xacro:property name="pi" value="3.1415"/>
@@ -39,3 +40,4 @@
         <origin xyz="0.05 0 0.85" rpy="0 1.5708 0"/>
     </xacro:epick_hand>
+    <xacro:robotiq_epick_gripper_transmission prefix="${prefix}"/>
 </robot>

File: pal_robotiq_epick_gripper/pal_robotiq_epick_description/urdf/robotiq_epick_model_macro.xacro (robot description, xacro)
@@ -1,5 +1,5 @@
 <?xml version="1.0"?>
 <robot xmlns:xacro="http://www.ros.org/wiki/xacro">
-  <xacro:include filename="$(find pal_robotiq_epick_description)/urdf/robotiq_epick.gazebo.xacro"/>
+  <xacro:include filename="$(find pal_robotiq_epick_description)/urdf/robotiq_epick_gripper.transmission.xacro" />
   <xacro:property name="joint_lower_limit" value="0.0" />
   <xacro:property name="joint_upper_limit" value="0.055" />
@@ -80,5 +80,5 @@
       </collision>  -->
     </link>
-    <joint name="${prefix}vacuum_joint" type="fixed">
+    <joint name="${prefix}finger_joint" type="fixed">
       <parent link="${prefix}base_link"/>
       <child link="${prefix}end_effector"/>
@@ -102,5 +102,5 @@
       </inertial>
     </link>
-  <!-- <xacro:epick_hand_gazebo robot_name="${robot_name}" />  -->
+    <xacro:robotiq_epick_gripper_transmission prefix="${prefix}"/>
   </xacro:macro>
 </robot>

Commit message: Add transmission folder and config files

File: pal_robotiq_epick_gripper/pal_robotiq_epick_description/robots/pal_robotiq_epick_gripper.urdf.xacro (robot description, xacro)
@@ -1,5 +1,5 @@
 <?xml version="1.0" ?>
 <robot name="robotiq_epick_gripper" xmlns:xacro="http://ros.org/wiki/xacro">
-    <xacro:include filename="$(find pal_robotiq_epick_description)/urdf/robotiq_epcick_gripper.transmission.xacro" />
+    <xacro:include filename="$(find pal_robotiq_epick_description)/urdf/robotiq_epick_gripper.transmission.xacro" />
     <xacro:include filename="$(find pal_robotiq_epick_description)/urdf/robotiq_epick_model_macro.xacro" />
     <xacro:property name="pi" value="3.1415"/>

File: pal_robotiq_epick_gripper/pal_robotiq_epick_description/urdf/robotiq_epick_model_macro.xacro (robot description, xacro)
@@ -80,8 +80,10 @@
       </collision>  -->
     </link>
-    <joint name="${prefix}finger_joint" type="fixed">
+    <joint name="${prefix}finger_joint" type="revolute">
       <parent link="${prefix}base_link"/>
       <child link="${prefix}end_effector"/>
       <origin xyz="0 0 ${0.13}" rpy="0 0 0"/>
+      <axis xyz="1 0 0" />
+      <limit lower="0" upper="1" velocity="2.0" effort="1000" />
     </joint>
     <link name="${prefix}end_effector">
