Commit message: Change joint name and configuration

File: pal_robotiq_epick_gripper/pal_robotiq_epick_description/urdf/robotiq_epick_gripper.transmission.xacro (robot description, xacro)
@@ -2,14 +2,12 @@
 <robot xmlns:xacro="http://ros.org/wiki/xacro">
   <xacro:macro name="robotiq_epick_gripper_transmission" params="prefix">
-    <transmission name="${prefix}finger_trans">
+    <transmission name="${prefix}vacuum_trans">
         <type>transmission_interface/SimpleTransmission</type>
-        <joint name="${prefix}finger_joint">
-            <hardwareInterface>hardware_interface/PositionJointInterface</hardwareInterface>
-            <hardwareInterface>hardware_interface/JointStateInterface</hardwareInterface>
+        <joint name="${prefix}vacuum_joint">
+            <hardwareInterface>hardware_interface/EffortJointInterface</hardwareInterface>
         </joint>
-        <actuator name="${prefix}motor">
+        <actuator name="${prefix}vacuum">
             <mechanicalReduction>1</mechanicalReduction>
-            <hardwareInterface>hardware_interface/PositionJointInterface</hardwareInterface>
-            <hardwareInterface>hardware_interface/JointStateInterface</hardwareInterface>
+            <hardwareInterface>hardware_interface/EffortJointInterface</hardwareInterface>
         </actuator>
     </transmission>

File: pal_robotiq_epick_gripper/pal_robotiq_epick_description/urdf/robotiq_epick_model_macro.xacro (robot description, xacro)
@@ -80,10 +80,10 @@
       </collision>  -->
     </link>
-    <joint name="${prefix}finger_joint" type="revolute">
+    <joint name="${prefix}vacuum_joint" type="prismatic">
       <parent link="${prefix}base_link"/>
       <child link="${prefix}end_effector"/>
       <origin xyz="0 0 ${0.13}" rpy="0 0 0"/>
       <axis xyz="1 0 0" />
-      <limit lower="0" upper="1" velocity="2.0" effort="1000" />
+      <limit lower="0" upper="0.01" velocity="2.0" effort="1000" />
     </joint>
     <link name="${prefix}end_effector">
