Commit message: add prefix for tiago dual

File: pal_robotiq_epick_gripper/pal_robotiq_epick_description/urdf/robotiq_epick_model_macro.xacro (robot description, xacro)
@@ -4,11 +4,11 @@
   <xacro:property name="joint_lower_limit" value="0.0" />
   <xacro:property name="joint_upper_limit" value="0.055" />
-  <xacro:macro name="epick_hand" params="hand_link_name robot_name parent">
-    <joint name="base_joint" type="fixed">
+  <xacro:macro name="epick_hand" params="hand_link_name robot_name prefix parent">
+    <joint name="${prefix}base_joint" type="fixed">
       <parent link="${parent}"/>
-      <child link="coupler_link"/>
+      <child link="${prefix}coupler_link"/>
       <origin xyz="0 0 0.0" rpy="${3.1416/2} 0 ${3.1416/2}"/>
     </joint>
-    <link name="coupler_link">
+    <link name="${prefix}coupler_link">
       <visual>
           <origin xyz="0 0 0.0" rpy="3.1416 0 0" />
@@ -34,10 +34,10 @@
       </inertial>
     </link>
-    <joint name="coupler_joint" type="fixed">
-      <parent link="coupler_link"/>
-      <child link="${hand_link_name}"/>
+    <joint name="${prefix}coupler_joint" type="fixed">
+      <parent link="${prefix}coupler_link"/>
+      <child link="${prefix}${hand_link_name}"/>
       <origin xyz="0 0 ${0.0273}" rpy="0 0 -${3.1416/2}"/>
     </joint>
-    <link name="${hand_link_name}">
+    <link name="${prefix}${hand_link_name}">
       <inertial>
         <mass value="0.745" />
@@ -80,10 +80,10 @@
       </collision>  -->
     </link>
-    <joint name="$hand__end_effector_joint" type="fixed">
-      <parent link="${hand_link_name}"/>
-      <child link="epick_end_effector"/>
+    <joint name="${prefix}${hand_link_name}_joint" type="fixed">
+      <parent link="${prefix}${hand_link_name}"/>
+      <child link="${prefix}epick_end_effector"/>
       <origin xyz="0 0 ${0.13}" rpy="0 0 0"/>
     </joint>
-    <link name="epick_end_effector">
+    <link name="${prefix}epick_end_effector">
       <gravity>0</gravity>
       <visual>

Commit message: Match the code with the other robotiq gripper + remove robot_name and hand_link_name unused parameters

File: pal_robotiq_epick_gripper/pal_robotiq_epick_description/urdf/robotiq_epick_model_macro.xacro (robot description, xacro)
@@ -4,9 +4,9 @@
   <xacro:property name="joint_lower_limit" value="0.0" />
   <xacro:property name="joint_upper_limit" value="0.055" />
-  <xacro:macro name="epick_hand" params="hand_link_name robot_name prefix parent">
+  <xacro:macro name="epick_hand" params="prefix parent *origin">
     <joint name="${prefix}base_joint" type="fixed">
       <parent link="${parent}"/>
       <child link="${prefix}coupler_link"/>
-      <origin xyz="0 0 0.0" rpy="${3.1416/2} 0 ${3.1416/2}"/>
+      <xacro:insert_block name="origin" />
     </joint>
     <link name="${prefix}coupler_link">
@@ -36,8 +36,8 @@
     <joint name="${prefix}coupler_joint" type="fixed">
       <parent link="${prefix}coupler_link"/>
-      <child link="${prefix}${hand_link_name}"/>
+      <child link="${prefix}base_link"/>
       <origin xyz="0 0 ${0.0273}" rpy="0 0 -${3.1416/2}"/>
     </joint>
-    <link name="${prefix}${hand_link_name}">
+    <link name="${prefix}base_link">
       <inertial>
         <mass value="0.745" />
@@ -80,10 +80,10 @@
       </collision>  -->
     </link>
-    <joint name="${prefix}${hand_link_name}_joint" type="fixed">
-      <parent link="${prefix}${hand_link_name}"/>
-      <child link="${prefix}epick_end_effector"/>
+    <joint name="${prefix}vacuum_joint" type="fixed">
+      <parent link="${prefix}base_link"/>
+      <child link="${prefix}end_effector"/>
       <origin xyz="0 0 ${0.13}" rpy="0 0 0"/>
     </joint>
-    <link name="${prefix}epick_end_effector">
+    <link name="${prefix}end_effector">
       <gravity>0</gravity>
       <visual>
@@ -102,5 +102,5 @@
       </inertial>
     </link>
-    <xacro:epick_hand_gazebo robot_name="${robot_name}" />
+  <!-- <xacro:epick_hand_gazebo robot_name="${robot_name}" />  -->
   </xacro:macro>
 </robot>

Commit message: Fix urdf for gazebo + change color ef the end effector

File: pal_robotiq_epick_gripper/pal_robotiq_epick_description/urdf/robotiq_epick_model_macro.xacro (robot description, xacro)
@@ -83,7 +83,8 @@
       <parent link="${prefix}base_link"/>
       <child link="${prefix}end_effector"/>
-      <origin xyz="0 0 ${0.13}" rpy="0 0 0"/>
-      <axis xyz="1 0 0" />
-      <limit lower="0" upper="0.01" velocity="2.0" effort="1000" />
+      <origin xyz="0 0 0.13" rpy="0 0 0"/>
+      <axis xyz="0 0 1" />
+      <limit lower="-0.01" upper="0.0" velocity="2.0" effort="1000"/>
+      <dynamics damping="0.1" friction="0.01"/>
     </joint>
     <link name="${prefix}end_effector">
@@ -94,7 +95,7 @@
           <cylinder radius="0.0225" length="0.01"/>
         </geometry>
-        <!-- <material name="transparent">
-          <color rgba="0 0 0 0"/>
-        </material> -->
+        <material name="transparent">
+          <color rgba="0.5 0.5 0.5 0.7"/>
+        </material>
       </visual>
       <inertial>

Commit message: Added grasping frame

File: pal_robotiq_epick_gripper/pal_robotiq_epick_description/urdf/robotiq_epick_model_macro.xacro (robot description, xacro)
@@ -105,4 +105,19 @@
       </inertial>
     </link>
+    <!-- Graping Frame -->
+    <joint name="${prefix}grasping_frame_joint" type="fixed">
+      <parent link="${prefix}base_link" />
+      <child link="${prefix}grasping_frame" />
+      <origin xyz="0 0 0.135" rpy="0 -1.5708 0" />
+    </joint>
+    <link name="${prefix}grasping_frame">
+      <inertial>
+        <origin xyz="0 0 0" rpy="0 0 0" />
+        <mass value="0.0001" />
+        <inertia ixx="0.00001" ixy="0.0" ixz="0.0"
+                iyy="0.00001" iyz="0.0"
+                izz="0.00001" />
+      </inertial>
+    </link>
     <xacro:robotiq_epick_gripper_transmission prefix="${prefix}"/>
   </xacro:macro>
