Commit message: added black material color to the coupling visual

File: pal_robotiq_85_gripper/pal_robotiq_85_description/urdf/robotiq_85_gripper.urdf.xacro (robot description, xacro)
@@ -236,4 +236,7 @@
   </xacro:macro>
   <xacro:macro name="pal_robotiq_coupling_link" params="prefix">
+    <material name="black">
+      <color rgba="0 0 0 1"/>
+    </material>
     <link name="${prefix}coupler_link">
         <visual>
@@ -243,4 +246,5 @@
                 <!--mesh filename="package://pal_robotiq_85_description/meshes/visual/pal_robotiq_coupling.stl"/-->
             </geometry>
+            <material name="black"/>
         </visual>
         <collision>

Commit message: Update URDF model with new meshes and some changes to mimic joints naming

File: pal_robotiq_85_gripper/pal_robotiq_85_description/urdf/robotiq_85_gripper.urdf.xacro (robot description, xacro)
@@ -176,5 +176,5 @@
     <gazebo>
       <!-- loading plugin: mimic joints works in gazebo now -->
-      <plugin filename="libroboticsgroup_gazebo_mimic_joint_plugin.so" name="${prefix}mimic_robotiq_85_1">
+      <plugin filename="libroboticsgroup_gazebo_mimic_joint_plugin.so" name="${prefix}${fingerprefix}mimic_robotiq_85_1">
         <joint>${prefix}finger_joint</joint>
         <mimicJoint>${prefix}${fingerprefix}_inner_knuckle_joint</mimicJoint>
@@ -195,5 +195,5 @@
     <gazebo>
       <!-- loading plugin: mimic joints works in gazebo now -->
-      <plugin filename="libroboticsgroup_gazebo_mimic_joint_plugin.so" name="${prefix}mimic_robotiq_85_4">
+      <plugin filename="libroboticsgroup_gazebo_mimic_joint_plugin.so" name="${prefix}${fingerprefix}mimic_robotiq_85_4">
         <joint>${prefix}finger_joint</joint>
         <mimicJoint>${prefix}${fingerprefix}_inner_finger_joint</mimicJoint>
@@ -219,7 +219,7 @@
       </inertial>
       <visual>
-        <origin xyz="0 0 0" rpy="0 0 0" />
-        <geometry>
-          <mesh filename="package://pal_robotiq_85_description/meshes/visual/robotiq_85_base_link.dae" scale="0.001 0.001 0.001"/>
+        <origin xyz="0 0 0" rpy="0 -1.5709 0" />
+        <geometry>
+          <mesh filename="package://pal_robotiq_85_description/meshes/visual/robotiq_85_base_link.stl"/>
         </geometry>
         <material name="">
@@ -234,4 +234,9 @@
       </collision>
     </link>
+    <gazebo reference="${prefix}base_link">
+      <mu1>0.9</mu1>
+      <mu2>0.9</mu2>
+      <material>Gazebo/Black</material>
+    </gazebo>
   </xacro:macro>
   <xacro:macro name="pal_robotiq_coupling_link" params="prefix">
@@ -261,4 +266,9 @@
         </inertial>
     </link>
+    <gazebo reference="${prefix}coupler_link">
+      <mu1>0.9</mu1>
+      <mu2>0.9</mu2>
+      <material>Gazebo/Black</material>
+    </gazebo>
   </xacro:macro>
   <xacro:macro name="pal_robotiq_coupling_joint" params="prefix parent *origin">

Commit message: more fixes+

File: pal_robotiq_85_gripper/pal_robotiq_85_description/urdf/robotiq_85_gripper.urdf.xacro (robot description, xacro)
@@ -2,9 +2,27 @@
 <robot xmlns:xacro="http://ros.org/wiki/xacro">
   <xacro:include filename="$(find pal_robotiq_85_description)/urdf/robotiq_85_gripper.transmission.xacro" />
+  <xacro:macro name="mimic_joint_plugin_gazebo" params="name_prefix parent_joint mimic_joint has_pid:=false multiplier:=1.0 offset:=0 sensitiveness:=0.0 max_effort:=10.0 robot_namespace:=''">
+    <gazebo>
+      <plugin name="${name_prefix}mimic_joint_plugin" filename="libroboticsgroup_gazebo_mimic_joint_plugin.so">
+        <joint>${parent_joint}</joint>
+        <mimicJoint>${mimic_joint}</mimicJoint>
+        <xacro:if value="${has_pid}">                     <!-- if set to true, PID parameters from "/gazebo_ros_control/pid_gains/${mimic_joint}" are loaded -->
+          <hasPID />
+        </xacro:if>
+        <multiplier>${multiplier}</multiplier>
+        <offset>${offset}</offset>
+        <sensitiveness>${sensitiveness}</sensitiveness>   <!-- if absolute difference between setpoint and process value is below this threshold, do nothing; 0.0 = disable [rad] -->
+        <maxEffort>${max_effort}</maxEffort>              <!-- only taken into account if has_pid:=true [Nm] -->
+        <xacro:unless value="${robot_namespace == ''}">
+          <robotNamespace>${robot_namespace}</robotNamespace>
+        </xacro:unless>
+      </plugin>
+    </gazebo>
+  </xacro:macro>
   <xacro:macro name="outer_knuckle" params="prefix fingerprefix ">
     <link name="${prefix}${fingerprefix}_outer_knuckle">
       <inertial>
         <origin xyz="-0.000200000000003065 0.0199435877845359 0.0292245259211331" rpy="0 0 0" />
-        <mass value="0.00853198276973456" />
+        <mass value="0.01853198276973456" />
         <inertia ixx="2.89328108496468E-06" ixy="-1.57935047237397E-19" ixz="-1.93980378593255E-19" iyy="1.86719750325683E-06" iyz="-1.21858577871576E-06" izz="1.21905238907251E-06" />
       </inertial>
@@ -174,13 +192,5 @@
       <mimic joint="${prefix}finger_joint" multiplier="1" offset="0" />
     </joint>
-    <gazebo>
-      <!-- loading plugin: mimic joints works in gazebo now -->
-      <plugin filename="libroboticsgroup_gazebo_mimic_joint_plugin.so" name="${prefix}${fingerprefix}mimic_robotiq_85_1">
-        <joint>${prefix}finger_joint</joint>
-        <mimicJoint>${prefix}${fingerprefix}_inner_knuckle_joint</mimicJoint>
-        <!--multiplier>1.0</multiplier>
-        <offset>0.0</offset-->
-      </plugin>
-    </gazebo>
+    <xacro:mimic_joint_plugin_gazebo name_prefix="${prefix}${fingerprefix}mimic_robotiq_85_1" parent_joint="${prefix}finger_joint" mimic_joint="${prefix}${fingerprefix}_inner_knuckle_joint" has_pid="false" multiplier="1.0" offset="0.0"/>
   </xacro:macro>
   <xacro:macro name="inner_finger_joint" params="prefix fingerprefix">
@@ -193,13 +203,5 @@
       <mimic joint="${prefix}finger_joint" multiplier="-1" offset="0" />
     </joint>
-    <gazebo>
-      <!-- loading plugin: mimic joints works in gazebo now -->
-      <plugin filename="libroboticsgroup_gazebo_mimic_joint_plugin.so" name="${prefix}${fingerprefix}mimic_robotiq_85_4">
-        <joint>${prefix}finger_joint</joint>
-        <mimicJoint>${prefix}${fingerprefix}_inner_finger_joint</mimicJoint>
-        <multiplier>-1.0</multiplier>
-        <offset>0.0</offset>
-      </plugin>
-    </gazebo>
+    <xacro:mimic_joint_plugin_gazebo name_prefix="${prefix}${fingerprefix}mimic_robotiq_85_4" parent_joint="${prefix}finger_joint" mimic_joint="${prefix}${fingerprefix}_inner_finger_joint" has_pid="false" multiplier="-1.0" offset="0.0"/>
   </xacro:macro>
   <xacro:macro name="inner_finger_pad_joint" params="prefix fingerprefix">
@@ -241,28 +243,28 @@
   </xacro:macro>
   <xacro:macro name="pal_robotiq_coupling_link" params="prefix">
+    <material name="black">
+      <color rgba="0 0 0 1"/>
+    </material>
     <link name="${prefix}coupler_link">
-      <material name="black">
-        <color rgba="0 0 0 1"/>
-      </material>
-        <visual>
-            <origin xyz="0 0 0.0" rpy="3.1416 0 0" />
-            <geometry>
-                <mesh filename="package://pal_robotiq_85_description/meshes/visual/pal_robotiq_coupling.stl"/>
-            </geometry>
-            <material name="black"/>
-        </visual>
-        <collision>
-            <origin xyz="0 0 0.0" rpy="3.1416 0 0" />
-            <geometry>
-                <mesh filename="package://pal_robotiq_85_description/meshes/visual/pal_robotiq_coupling.stl"/>
-            </geometry>
-        </collision>
-        <inertial>
-            <mass value="0.1" />
-            <origin xyz="0.0 0.0 0.0" />
-            <inertia ixx = "0.000001" ixy = "0.000000" ixz = "0.000000"
-                     iyx = "0.000000" iyy = "0.000001" iyz = "0.000000"
-                     izx = "0.000000" izy = "0.000000" izz = "0.000001" />
-        </inertial>
+      <visual>
+          <origin xyz="0 0 0.0" rpy="3.1416 0 0" />
+          <geometry>
+              <mesh filename="package://pal_robotiq_85_description/meshes/visual/pal_robotiq_coupling.stl"/>
+          </geometry>
+          <material name="black"/>
+      </visual>
+      <collision>
+          <origin xyz="0 0 0.0" rpy="3.1416 0 0" />
+          <geometry>
+              <mesh filename="package://pal_robotiq_85_description/meshes/visual/pal_robotiq_coupling.stl"/>
+          </geometry>
+      </collision>
+      <inertial>
+          <mass value="0.2" />
+          <origin xyz="0.0 0.0 -0.01" />
+          <inertia ixx = "0.000001" ixy = "0.000000" ixz = "0.000000"
+                   iyx = "0.000000" iyy = "0.000001" iyz = "0.000000"
+                   izx = "0.000000" izy = "0.000000" izz = "0.000001" />
+      </inertial>
     </link>
     <gazebo reference="${prefix}coupler_link">
@@ -317,14 +319,6 @@
       <limit lower="0" upper="0.81" velocity="2.0" effort="1000" />
       <mimic joint="${prefix}finger_joint" multiplier="1" offset="0" />
-      <gazebo>
-        <!-- loading plugin: mimic joints works in gazebo now -->
-        <plugin filename="libroboticsgroup_gazebo_mimic_joint_plugin.so" name="${prefix}mimic_robotiq_85_3">
-            <joint>${prefix}finger_joint</joint>
-            <mimicJoint>${prefix}right_outer_knuckle_joint</mimicJoint>
-            <!--multiplier>1.0</multiplier>
-            <offset>0.0</offset-->
-        </plugin>
-      </gazebo>
-    </joint>
+    </joint>
+    <xacro:mimic_joint_plugin_gazebo name_prefix="${prefix}mimic_robotiq_85_3" parent_joint="${prefix}finger_joint" mimic_joint="${prefix}right_outer_knuckle_joint" has_pid="false" multiplier="1.0" offset="0.0"/>
     <xacro:finger_joints prefix="${prefix}" fingerprefix="right" reflect="-1.0"/>
   </xacro:macro>

Commit message: Update inertias of the links to a proper functional one

File: pal_robotiq_85_gripper/pal_robotiq_85_description/urdf/robotiq_85_gripper.urdf.xacro (robot description, xacro)
@@ -20,10 +20,10 @@
     </gazebo>
   </xacro:macro>
-  <xacro:macro name="outer_knuckle" params="prefix fingerprefix ">
+  <xacro:macro name="outer_knuckle" params="prefix fingerprefix reflect">
     <link name="${prefix}${fingerprefix}_outer_knuckle">
       <inertial>
-        <origin xyz="-0.000200000000003065 0.0199435877845359 0.0292245259211331" rpy="0 0 0" />
-        <mass value="0.01853198276973456" />
-        <inertia ixx="2.89328108496468E-06" ixy="-1.57935047237397E-19" ixz="-1.93980378593255E-19" iyy="1.86719750325683E-06" iyz="-1.21858577871576E-06" izz="1.21905238907251E-06" />
+        <origin xyz="${reflect * 0.01545} 0 -0.00118" rpy="0 0 0" />
+        <mass value="0.01252" />
+        <inertia ixx="312.44E-9" ixy="0" ixz="-168.09E-9" iyy="2156E-9" iyz="0" izz="2027.51E-9" />
       </inertial>
       <visual>
@@ -51,10 +51,10 @@
     </gazebo>
   </xacro:macro>
-  <xacro:macro name="outer_finger" params="prefix fingerprefix ">
+  <xacro:macro name="outer_finger" params="prefix fingerprefix reflect">
     <link name="${prefix}${fingerprefix}_outer_finger">
       <inertial>
-        <origin xyz="0.00030115855001899 0.0373907951953854 -0.0208027427000385" rpy="0 0 0" />
-        <mass value="0.022614240507152" />
-        <inertia ixx="1.52518312458174E-05" ixy="9.76583423954399E-10" ixz="-5.43838577022588E-10" iyy="6.17694243867776E-06" iyz="6.78636130740228E-06" izz="1.16494917907219E-05" />
+        <origin xyz="0.004 0 ${reflect * 0.01892}" rpy="0 0 0" />
+        <mass value="0.03848" />
+        <inertia ixx="12341E-9" ixy="0" ixz="-2152.21E-9" iyy="10617E-9" iyz="0" izz="4812.09E-9" />
       </inertial>
       <visual>
@@ -82,10 +82,10 @@
     </gazebo>
   </xacro:macro>
-  <xacro:macro name="inner_knuckle" params="prefix fingerprefix ">
+  <xacro:macro name="inner_knuckle" params="prefix fingerprefix reflect">
     <link name="${prefix}${fingerprefix}_inner_knuckle">
       <inertial>
-        <origin xyz="0.000123011831763771 0.0507850843201817 0.00103968640075166" rpy="0 0 0" />
-       <mass value="0.0271177346495152" />
-        <inertia ixx="2.61910379223783E-05" ixy="-2.43616858946494E-07" ixz="-6.37789906117123E-09" iyy="2.8270243746167E-06" iyz="-5.37200748039765E-07" izz="2.83695868220296E-05" />
+        <origin xyz="${reflect * 0.01952} 0 0.022" rpy="0 0 0" />
+        <mass value="0.02731" />
+        <inertia ixx="8621.3E-9" ixy="0" ixz="-3646.49E-9" iyy="8004.28E-9" iyz="0" izz="7704.42E-9" />
       </inertial>
       <visual>
@@ -113,10 +113,10 @@
     </gazebo>
   </xacro:macro>
-  <xacro:macro name="inner_finger" params="prefix fingerprefix ">
+  <xacro:macro name="inner_finger" params="prefix fingerprefix reflect">
     <link name="${prefix}${fingerprefix}_inner_finger">
       <inertial>
-        <origin xyz="0.000299999999999317 0.0160078233491243 -0.0136945669206257" rpy="0 0 0" />
-        <mass value="0.0104003125914103" />
-        <inertia ixx="2.71909453810972E-06" ixy="1.35402465472579E-21" ixz="-7.1817349065269E-22" iyy="7.69100314106116E-07" iyz="6.74715432769696E-07" izz="2.30315190420171E-06" />
+        <origin xyz="${reflect * -0.01409} 0 0.01569" rpy="0 0 0" />
+        <mass value="0.037" />
+        <inertia ixx="12446.57E-9" ixy="0" ixz="4167.81E-9" iyy="14201.18E-9" iyz="0" izz="4979.86E-9" />
       </inertial>
       <visual>
@@ -216,7 +216,7 @@
     <link name="${prefix}base_link">
       <inertial>
-        <origin xyz="8.625E-08 -4.6583E-06 0.03145" rpy="0 0 0" />
-        <mass value="0.22652" />
-        <inertia ixx="0.00020005" ixy="-4.2442E-10" ixz="-2.9069E-10" iyy="0.00017832" iyz="-3.4402E-08" izz="0.00013478" />
+        <origin xyz="-0.00013 -0.00011 0.03284" rpy="0 0 0" />
+        <mass value="0.55938" />
+        <inertia ixx="605783E-9" ixy="-579.95E-9" ixz="2765.53E-9" iyy="720148E-9" iyz="618E-9" izz="510534E-9" />
       </inertial>
       <visual>
@@ -294,10 +294,10 @@
     <xacro:inner_finger_pad_joint prefix="${prefix}" fingerprefix="${fingerprefix}"/>
   </xacro:macro>
-  <xacro:macro name="finger_links" params="prefix fingerprefix">
-    <xacro:outer_knuckle prefix="${prefix}" fingerprefix="${fingerprefix}" />
-    <xacro:outer_finger prefix="${prefix}" fingerprefix="${fingerprefix}" />
-    <xacro:inner_finger prefix="${prefix}" fingerprefix="${fingerprefix}" />
+  <xacro:macro name="finger_links" params="prefix fingerprefix reflect">
+    <xacro:outer_knuckle prefix="${prefix}" fingerprefix="${fingerprefix}" reflect="${reflect}"/>
+    <xacro:outer_finger prefix="${prefix}" fingerprefix="${fingerprefix}" reflect="${reflect}"/>
+    <xacro:inner_finger prefix="${prefix}" fingerprefix="${fingerprefix}" reflect="${reflect}"/>
     <xacro:inner_finger_pad prefix="${prefix}" fingerprefix="${fingerprefix}"/>
-    <xacro:inner_knuckle prefix="${prefix}" fingerprefix="${fingerprefix}" />
+    <xacro:inner_knuckle prefix="${prefix}" fingerprefix="${fingerprefix}" reflect="${reflect}"/>
   </xacro:macro>
   <xacro:macro name="finger_joint" params="prefix">
@@ -327,6 +327,6 @@
     <xacro:robotiq_base_link prefix="${prefix}"/>
     <xacro:pal_robotiq_coupling_link prefix="${prefix}"/>
-    <xacro:finger_links prefix="${prefix}" fingerprefix="left" />
-    <xacro:finger_links prefix="${prefix}" fingerprefix="right"/>
+    <xacro:finger_links prefix="${prefix}" fingerprefix="left" reflect="1"/>
+    <xacro:finger_links prefix="${prefix}" fingerprefix="right" reflect="-1"/>
     <xacro:robotiq_base_joint prefix="${prefix}" />
     <xacro:pal_robotiq_coupling_joint prefix="${prefix}" parent="${parent}">

Commit message: fix the issue with the inner_finger link on wrong limits

File: pal_robotiq_85_gripper/pal_robotiq_85_description/urdf/robotiq_85_gripper.urdf.xacro (robot description, xacro)
@@ -200,5 +200,5 @@
       <child link="${prefix}${fingerprefix}_inner_finger" />
       <axis xyz="1 0 0" />
-      <limit lower="0" upper="0.8757" velocity="2.0" effort="1000" />
+      <limit lower="-0.8757" upper="0" velocity="2.0" effort="1000" />
       <mimic joint="${prefix}finger_joint" multiplier="-1" offset="0" />
     </joint>

Commit message: update the base link visual STL

File: pal_robotiq_85_gripper/pal_robotiq_85_description/urdf/robotiq_85_gripper.urdf.xacro (robot description, xacro)
@@ -221,7 +221,7 @@
       </inertial>
       <visual>
-        <origin xyz="0 0 0" rpy="0 -1.5709 0" />
-        <geometry>
-          <mesh filename="package://pal_robotiq_85_description/meshes/visual/robotiq_85_base_link.stl"/>
+        <origin xyz="0 0 0" rpy="0 0 0" />
+        <geometry>
+          <mesh filename="package://pal_robotiq_85_description/meshes/visual/robotiq_base_link.stl"/>
         </geometry>
         <material name="">

Commit message: Update inertia parameters of base link of robotiq-2f-85

File: pal_robotiq_85_gripper/pal_robotiq_85_description/urdf/robotiq_85_gripper.urdf.xacro (robot description, xacro)
@@ -218,7 +218,7 @@
     <link name="${prefix}base_link">
       <inertial>
-        <origin xyz="-0.00013 -0.00011 0.03284" rpy="0 0 0" />
-        <mass value="0.55938" />
-        <inertia ixx="605783E-9" ixy="-579.95E-9" ixz="2765.53E-9" iyy="720148E-9" iyz="618E-9" izz="510534E-9" />
+        <origin xyz="8.625E-08 -4.6583E-06 0.03145" rpy="0 0 0" />
+        <mass value="0.22652" />
+        <inertia ixx="0.00020005" ixy="-4.2442E-10" ixz="-2.9069E-10" iyy="0.00017832" iyz="-3.4402E-08" izz="0.00013478" />
       </inertial>
       <visual>
@@ -234,5 +234,5 @@
         <origin xyz="0 0 0" rpy="0 0 0" />
         <geometry>
-           <mesh filename="package://pal_robotiq_85_description/meshes/collision/robotiq_base_link.stl" />
+          <mesh filename="package://pal_robotiq_85_description/meshes/collision/robotiq_base_link.stl" />
         </geometry>
       </collision>

Commit message: Tweak damping parameter because of ABORTED error with play_motion

File: pal_robotiq_85_gripper/pal_robotiq_85_description/urdf/robotiq_85_gripper.urdf.xacro (robot description, xacro)
@@ -196,8 +196,4 @@
       <axis xyz="1 0 0" />
     </joint>
-    <gazebo reference="${prefix}${fingerprefix}_outer_finger_joint">
-      <provideFeedback>1</provideFeedback>
-      <implicitSpringDamper>1</implicitSpringDamper>
-    </gazebo>
   </xacro:macro>
   <xacro:macro name="inner_knuckle_joint" params="prefix fingerprefix reflect">
@@ -208,5 +204,5 @@
       <child link="${prefix}${fingerprefix}_inner_knuckle" />
       <axis xyz="1 0 0" />
-      <limit lower="0" upper="0.8757" velocity="0.5" effort="0.05" />
+      <limit lower="0" upper="0.8757" velocity="2" effort="0.05" />
       <mimic joint="${prefix}finger_joint" multiplier="1" offset="0" />
     </joint>
@@ -219,5 +215,5 @@
       <child link="${prefix}${fingerprefix}_inner_finger" />
       <axis xyz="1 0 0" />
-      <limit lower="-0.8757" upper="0" velocity="0.5" effort="0.05" />
+      <limit lower="-0.8757" upper="0" velocity="2" effort="0.05" />
       <mimic joint="${prefix}finger_joint" multiplier="-1" offset="0" />
     </joint>
@@ -323,6 +319,6 @@
       <child link="${prefix}left_outer_knuckle" />
       <axis xyz="1 0 0" />
-      <limit lower="0" upper="0.8" velocity="0.5" effort="0.05" />
-      <dynamics damping="0.2"/>
+      <limit lower="0" upper="0.8" velocity="2" effort="0.05" />
+      <dynamics damping="0.03"/>
     </joint>
     <gazebo reference="${prefix}finger_joint">
@@ -338,5 +334,5 @@
       <child link="${prefix}right_outer_knuckle" />
       <axis xyz="1 0 0" />
-      <limit lower="0" upper="0.81" velocity="0.5" effort="0.05" />
+      <limit lower="0" upper="0.81" velocity="2" effort="0.05" />
       <mimic joint="${prefix}finger_joint" multiplier="1" offset="0" />
     </joint>
