Commit message: Improve is_grasped topic in simulation

File: pal_robotiq_85_gripper/pal_robotiq_85_description/urdf/robotiq_85_gripper.urdf.xacro (robot description, xacro)
@@ -4,5 +4,5 @@
   <xacro:property name="finger_joint_damping" value="0.0025"/>
   <xacro:property name="finger_joint_friction" value="0.0"/>
-  <xacro:macro name="mimic_joint_plugin_gazebo" params="name_prefix parent_joint mimic_joint has_pid:=false multiplier:=1.0 offset:=0 sensitiveness:=0.0 max_effort:=0.05 robot_namespace:=''">
+  <xacro:macro name="mimic_joint_plugin_gazebo" params="name_prefix parent_joint mimic_joint has_pid:=false multiplier:=1.0 offset:=0 sensitiveness:=0.0 max_effort:=0.1 robot_namespace:=''">
     <gazebo>
       <plugin name="${name_prefix}mimic_joint_plugin" filename="libroboticsgroup_upatras_gazebo_mimic_joint_plugin.so">
@@ -105,8 +105,8 @@
       <kp>1000000.0</kp>
       <kd>100.0</kd>
-      <mu1>1000.0</mu1>
-      <mu2>1000.0</mu2>
+      <mu1>Inf</mu1>
+      <mu2>Inf</mu2>
       <fdir1>0 0 0</fdir1>
-      <maxVel>1.0</maxVel>
+      <maxVel>0.0</maxVel>
       <minDepth>0.01</minDepth>
       <material>Gazebo/DarkGrey</material>
@@ -139,11 +139,28 @@
     </link>
     <gazebo reference="${prefix}${fingerprefix}_inner_finger">
+      <collision name="${prefix}${fingerprefix}_inner_finger">
+        <surface>
+          <friction>
+            <torsional>
+              <coefficient>10.0</coefficient>
+              <use_patch_radius>true</use_patch_radius>
+              <patch_radius>0.05</patch_radius>
+            </torsional>
+          </friction>
+          <contact>
+            <poissons_ratio>0.5</poissons_ratio>
+            <elastic_modulus>1e8</elastic_modulus>
+          </contact>
+        </surface>
+      </collision>
+      <mu1>Inf</mu1>
+      <mu2>Inf</mu2>
+      <maxVel>0.0</maxVel>
       <kp>1000000.0</kp>
       <kd>100.0</kd>
-      <mu1>1000.0</mu1>
-      <mu2>1000.0</mu2>
-      <fdir1>0 0 0</fdir1>
-      <maxVel>1.0</maxVel>
+      <fdir1>1 0 0</fdir1>
+      <maxVel>0.0</maxVel>
       <minDepth>0.01</minDepth>
+      <maxContacts>100</maxContacts>
       <material>Gazebo/DarkGrey</material>
     </gazebo>
@@ -178,14 +195,4 @@
       </inertial>
     </link>
-    <gazebo reference="${prefix}${fingerprefix}_inner_finger_pad">
-      <kp>1000000.0</kp>
-      <kd>100.0</kd>
-      <mu1>1000.0</mu1>
-      <mu2>1000.0</mu2>
-      <fdir1>0 0 0</fdir1>
-      <maxVel>1.0</maxVel>
-      <minDepth>0.01</minDepth>
-      <material>Gazebo/DarkGrey</material>
-    </gazebo>
   </xacro:macro>
   <xacro:macro name="outer_finger_joint" params="prefix fingerprefix">
@@ -204,5 +211,5 @@
       <child link="${prefix}${fingerprefix}_inner_knuckle" />
       <axis xyz="1 0 0" />
-      <limit lower="0" upper="0.8757" velocity="2" effort="0.05" />
+      <limit lower="0" upper="0.8757" velocity="2" effort="0.1" />
       <mimic joint="${prefix}finger_joint" multiplier="1" offset="0" />
     </joint>
@@ -215,5 +222,5 @@
       <child link="${prefix}${fingerprefix}_inner_finger" />
       <axis xyz="1 0 0" />
-      <limit lower="-0.8757" upper="0" velocity="2" effort="0.05" />
+      <limit lower="-0.8757" upper="0" velocity="2" effort="0.1" />
       <mimic joint="${prefix}finger_joint" multiplier="-1" offset="0" />
     </joint>
@@ -336,5 +343,5 @@
       <child link="${prefix}left_outer_knuckle" />
       <axis xyz="1 0 0" />
-      <limit lower="0" upper="0.8" velocity="2" effort="0.05" />
+      <limit lower="0" upper="0.8" velocity="2" effort="0.1" />
       <dynamics damping="0.03"/>
     </joint>
@@ -351,5 +358,5 @@
       <child link="${prefix}right_outer_knuckle" />
       <axis xyz="1 0 0" />
-      <limit lower="0" upper="0.81" velocity="2" effort="0.05" />
+      <limit lower="0" upper="0.81" velocity="2" effort="0.1" />
       <mimic joint="${prefix}finger_joint" multiplier="1" offset="0" />
     </joint>

Commit message: improve gripper grasping frame position for 2f-85

File: pal_robotiq_85_gripper/pal_robotiq_85_description/urdf/robotiq_85_gripper.urdf.xacro (robot description, xacro)
@@ -291,5 +291,5 @@
       <parent link="${prefix}base_link" />
       <child link="${prefix}grasping_frame" />
-      <origin xyz="0 0 0.12" rpy="0 -1.5708 0" />
+      <origin xyz="0 0 0.10" rpy="0 -1.5708 0" />
     </joint>
     <link name="${prefix}grasping_frame">
