Commit message: Fix the URDF of 140 model the mimic configuration

File: pal_robotiq_140_gripper/pal_robotiq_140_description/urdf/robotiq_140_gripper.urdf.xacro (robot description, xacro)
@@ -2,4 +2,22 @@
 <robot xmlns:xacro="http://ros.org/wiki/xacro">
   <xacro:include filename="$(find pal_robotiq_140_description)/urdf/robotiq_140_gripper.transmission.xacro" />
+  <xacro:macro name="mimic_joint_plugin_gazebo" params="name_prefix parent_joint mimic_joint has_pid:=false multiplier:=1.0 offset:=0 sensitiveness:=0.0 max_effort:=10.0 robot_namespace:=''">
+    <gazebo>
+      <plugin name="${name_prefix}mimic_joint_plugin" filename="libroboticsgroup_gazebo_mimic_joint_plugin.so">
+        <joint>${parent_joint}</joint>
+        <mimicJoint>${mimic_joint}</mimicJoint>
+        <xacro:if value="${has_pid}">                     <!-- if set to true, PID parameters from "/gazebo_ros_control/pid_gains/${mimic_joint}" are loaded -->
+          <hasPID />
+        </xacro:if>
+        <multiplier>${multiplier}</multiplier>
+        <offset>${offset}</offset>
+        <sensitiveness>${sensitiveness}</sensitiveness>   <!-- if absolute difference between setpoint and process value is below this threshold, do nothing; 0.0 = disable [rad] -->
+        <maxEffort>${max_effort}</maxEffort>              <!-- only taken into account if has_pid:=true [Nm] -->
+        <xacro:unless value="${robot_namespace == ''}">
+          <robotNamespace>${robot_namespace}</robotNamespace>
+        </xacro:unless>
+      </plugin>
+    </gazebo>
+  </xacro:macro>
   <xacro:macro name="outer_knuckle" params="prefix fingerprefix stroke">
     <link name="${prefix}${fingerprefix}_outer_knuckle">
@@ -181,13 +199,5 @@
       <mimic joint="${prefix}finger_joint" multiplier="-1" offset="0" />
     </joint>
-    <gazebo>
-      <!-- loading plugin: mimic joints works in gazebo now -->
-      <plugin filename="libroboticsgroup_gazebo_mimic_joint_plugin.so" name="${prefix}mimic_robotiq_85_1">
-        <joint>${prefix}finger_joint</joint>
-        <mimicJoint>${prefix}${fingerprefix}_inner_knuckle_joint</mimicJoint>
-        <!--multiplier>1.0</multiplier>
-        <offset>0.0</offset-->
-      </plugin>
-    </gazebo>
+    <xacro:mimic_joint_plugin_gazebo name_prefix="${prefix}${fingerprefix}mimic_robotiq_85_1" parent_joint="${prefix}finger_joint" mimic_joint="${prefix}${fingerprefix}_inner_knuckle_joint" has_pid="false" multiplier="-1.0" offset="0.0"/>
   </xacro:macro>
   <xacro:macro name="inner_finger_joint" params="prefix fingerprefix">
@@ -200,13 +210,5 @@
       <mimic joint="${prefix}finger_joint" multiplier="1" offset="0" />
     </joint>
-    <gazebo>
-      <!-- loading plugin: mimic joints works in gazebo now -->
-      <plugin filename="libroboticsgroup_gazebo_mimic_joint_plugin.so" name="${prefix}mimic_robotiq_85_4">
-        <joint>${prefix}finger_joint</joint>
-        <mimicJoint>${prefix}${fingerprefix}_inner_finger_joint</mimicJoint>
-        <multiplier>-1.0</multiplier>
-        <offset>0.0</offset>
-      </plugin>
-    </gazebo>
+    <xacro:mimic_joint_plugin_gazebo name_prefix="${prefix}${fingerprefix}mimic_robotiq_85_1" parent_joint="${prefix}finger_joint" mimic_joint="${prefix}${fingerprefix}_inner_finger_joint" has_pid="false" multiplier="1.0" offset="0.0"/>
   </xacro:macro>
   <xacro:macro name="inner_finger_pad_joint" params="prefix fingerprefix">
@@ -281,4 +283,5 @@
     <mimic joint="${prefix}finger_joint" multiplier="-1" offset="0" />
     </joint>
+    <xacro:mimic_joint_plugin_gazebo name_prefix="${prefix}mimic_robotiq_85_5" parent_joint="${prefix}finger_joint" mimic_joint="${prefix}right_outer_knuckle_joint" has_pid="false" multiplier="-1.0" offset="0.0"/>
     <xacro:finger_joints prefix="${prefix}" fingerprefix="right" reflect="-1.0"/>
   </xacro:macro>

Commit message: Update the gazebo material types

File: pal_robotiq_140_gripper/pal_robotiq_140_description/urdf/robotiq_140_gripper.urdf.xacro (robot description, xacro)
@@ -46,9 +46,10 @@
     </link>
     <gazebo reference="${prefix}${fingerprefix}_outer_knuckle">
-        <implicitSpringDamper>1</implicitSpringDamper>
-        <mu1>100000</mu1>
-        <mu2>100000</mu2>
-        <kp>100000000.0</kp>
-        <kd>1.0</kd>
+      <implicitSpringDamper>1</implicitSpringDamper>
+      <mu1>100000</mu1>
+      <mu2>100000</mu2>
+      <kp>100000000.0</kp>
+      <kd>1.0</kd>
+      <material>Gazebo/Black</material>
     </gazebo>
   </xacro:macro>
@@ -79,9 +80,10 @@
     </link>
     <gazebo reference="{prefix}${fingerprefix}_outer_finger">
-        <implicitSpringDamper>1</implicitSpringDamper>
-        <mu1>100000</mu1>
-        <mu2>100000</mu2>
-        <kp>100000000.0</kp>
-        <kd>1.0</kd>
+      <implicitSpringDamper>1</implicitSpringDamper>
+      <mu1>100000</mu1>
+      <mu2>100000</mu2>
+      <kp>100000000.0</kp>
+      <kd>1.0</kd>
+      <material>Gazebo/Black</material>
     </gazebo>
   </xacro:macro>
@@ -112,9 +114,10 @@
     </link>
     <gazebo reference="${prefix}${fingerprefix}_inner_knuckle">
-        <implicitSpringDamper>1</implicitSpringDamper>
-        <mu1>100000</mu1>
-        <mu2>100000</mu2>
-        <kp>100000000.0</kp>
-        <kd>1.0</kd>
+      <implicitSpringDamper>1</implicitSpringDamper>
+      <mu1>100000</mu1>
+      <mu2>100000</mu2>
+      <kp>100000000.0</kp>
+      <kd>1.0</kd>
+      <material>Gazebo/Black</material>
     </gazebo>
   </xacro:macro>
@@ -145,9 +148,10 @@
     </link>
     <gazebo reference="${prefix}${fingerprefix}_inner_finger">
-        <implicitSpringDamper>1</implicitSpringDamper>
-        <mu1>100000</mu1>
-        <mu2>100000</mu2>
-        <kp>100000000.0</kp>
-        <kd>1.0</kd>
+      <implicitSpringDamper>1</implicitSpringDamper>
+      <mu1>100000</mu1>
+      <mu2>100000</mu2>
+      <kp>100000000.0</kp>
+      <kd>1.0</kd>
+      <material>Gazebo/Black</material>
     </gazebo>
   </xacro:macro>
@@ -175,9 +179,10 @@
     </link>
     <gazebo reference="${prefix}${fingerprefix}_inner_finger_pad">
-        <implicitSpringDamper>1</implicitSpringDamper>
-        <mu1>100000</mu1>
-        <mu2>100000</mu2>
-        <kp>100000000.0</kp>
-        <kd>1.0</kd>
+      <implicitSpringDamper>1</implicitSpringDamper>
+      <mu1>100000</mu1>
+      <mu2>100000</mu2>
+      <kp>100000000.0</kp>
+      <kd>1.0</kd>
+      <material>Gazebo/DarkGrey</material>
     </gazebo>
   </xacro:macro>
@@ -243,4 +248,9 @@
       </collision>
     </link>
+    <gazebo reference="${prefix}base_link">
+      <mu1>0.9</mu1>
+      <mu2>0.9</mu2>
+      <material>Gazebo/Black</material>
+    </gazebo>
   </xacro:macro>
   <xacro:macro name="pal_robotiq_coupling_link" params="prefix">

File: pal_robotiq_85_gripper/pal_robotiq_85_description/urdf/robotiq_85_gripper.urdf.xacro (robot description, xacro)
@@ -49,4 +49,5 @@
         <kp>100000000.0</kp>
         <kd>1.0</kd>
+        <material>Gazebo/DarkGrey</material>
     </gazebo>
   </xacro:macro>
@@ -153,5 +154,5 @@
         </geometry>
         <material name="">
-          <color rgba="0.9 0.9 0.9 1" />
+          <color rgba="0. 0. 0. 1" />
         </material>
       </visual>
@@ -167,9 +168,10 @@
     </link>
     <gazebo reference="${prefix}${fingerprefix}_inner_finger_pad">
-        <implicitSpringDamper>1</implicitSpringDamper>
-        <mu1>100000</mu1>
-        <mu2>100000</mu2>
-        <kp>100000000.0</kp>
-        <kd>1.0</kd>
+      <implicitSpringDamper>1</implicitSpringDamper>
+      <mu1>100000</mu1>
+      <mu2>100000</mu2>
+      <kp>100000000.0</kp>
+      <kd>1.0</kd>
+      <material>Gazebo/DarkGrey</material>
     </gazebo>
   </xacro:macro>
@@ -243,7 +245,4 @@
   </xacro:macro>
   <xacro:macro name="pal_robotiq_coupling_link" params="prefix">
-    <material name="black">
-      <color rgba="0 0 0 1"/>
-    </material>
     <link name="${prefix}coupler_link">
       <visual>
@@ -252,5 +251,7 @@
               <mesh filename="package://pal_robotiq_85_description/meshes/visual/pal_robotiq_coupling.stl"/>
           </geometry>
-          <material name="black"/>
+          <material name="black">
+            <color rgba="0 0 0 1"/>
+          </material>
       </visual>
       <collision>

Commit message: fix the black material not unique issue

File: pal_robotiq_140_gripper/pal_robotiq_140_description/urdf/robotiq_140_gripper.urdf.xacro (robot description, xacro)
@@ -255,7 +255,4 @@
   </xacro:macro>
   <xacro:macro name="pal_robotiq_coupling_link" params="prefix">
-    <material name="black">
-      <color rgba="0 0 0 1"/>
-    </material>
     <link name="${prefix}coupler_link">
       <visual>
@@ -264,5 +261,7 @@
               <mesh filename="package://pal_robotiq_85_description/meshes/visual/pal_robotiq_coupling.stl"/>
           </geometry>
-          <material name="black"/>
+          <material name="">
+            <color rgba="0 0 0 1"/>
+          </material>
       </visual>
       <collision>

File: pal_robotiq_85_gripper/pal_robotiq_85_description/urdf/robotiq_85_gripper.urdf.xacro (robot description, xacro)
@@ -251,5 +251,5 @@
               <mesh filename="package://pal_robotiq_85_description/meshes/visual/pal_robotiq_coupling.stl"/>
           </geometry>
-          <material name="black">
+          <material name="">
             <color rgba="0 0 0 1"/>
           </material>
