Commit message: Update the version of the mimicjoint + update the center of mass and inertia of the robotiq 85 gripper + adapt the force and collision in gazebo to grasp objects

File: pal_robotiq_140_gripper/pal_robotiq_140_description/urdf/robotiq_140_gripper.urdf.xacro (robot description, xacro)
@@ -2,7 +2,9 @@
 <robot xmlns:xacro="http://ros.org/wiki/xacro">
   <xacro:include filename="$(find pal_robotiq_140_description)/urdf/robotiq_140_gripper.transmission.xacro" />
-  <xacro:macro name="mimic_joint_plugin_gazebo" params="name_prefix parent_joint mimic_joint has_pid:=false multiplier:=1.0 offset:=0 sensitiveness:=0.0 max_effort:=10.0 robot_namespace:=''">
+  <xacro:property name="finger_joint_damping" value="0.0025"/>
+  <xacro:property name="finger_joint_friction" value="0.0"/>
+  <xacro:macro name="mimic_joint_plugin_gazebo" params="name_prefix parent_joint mimic_joint has_pid:=false multiplier:=1.0 offset:=0 sensitiveness:=0.0 max_effort:=0.05 robot_namespace:=''">
     <gazebo>
-      <plugin name="${name_prefix}mimic_joint_plugin" filename="libroboticsgroup_gazebo_mimic_joint_plugin.so">
+      <plugin name="${name_prefix}mimic_joint_plugin" filename="libroboticsgroup_upatras_gazebo_mimic_joint_plugin.so">
         <joint>${parent_joint}</joint>
         <mimicJoint>${mimic_joint}</mimicJoint>
@@ -45,12 +47,4 @@
       </collision>
     </link>
-    <gazebo reference="${prefix}${fingerprefix}_outer_knuckle">
-      <implicitSpringDamper>1</implicitSpringDamper>
-      <mu1>100000</mu1>
-      <mu2>100000</mu2>
-      <kp>100000000.0</kp>
-      <kd>1.0</kd>
-      <material>Gazebo/Black</material>
-    </gazebo>
   </xacro:macro>
   <xacro:macro name="outer_finger" params="prefix fingerprefix stroke">
@@ -79,11 +73,6 @@
       </collision>
     </link>
-    <gazebo reference="{prefix}${fingerprefix}_outer_finger">
-      <implicitSpringDamper>1</implicitSpringDamper>
-      <mu1>100000</mu1>
-      <mu2>100000</mu2>
-      <kp>100000000.0</kp>
-      <kd>1.0</kd>
-      <material>Gazebo/Black</material>
+    <gazebo reference="${prefix}${fingerprefix}_outer_finger">
+      <material>Gazebo/DarkGrey</material>
     </gazebo>
   </xacro:macro>
@@ -114,10 +103,12 @@
     </link>
     <gazebo reference="${prefix}${fingerprefix}_inner_knuckle">
-      <implicitSpringDamper>1</implicitSpringDamper>
-      <mu1>100000</mu1>
-      <mu2>100000</mu2>
-      <kp>100000000.0</kp>
-      <kd>1.0</kd>
-      <material>Gazebo/Black</material>
+      <kp>1000000.0</kp>
+      <kd>100.0</kd>
+      <mu1>1000.0</mu1>
+      <mu2>1000.0</mu2>
+      <fdir1>0 0 0</fdir1>
+      <maxVel>1.0</maxVel>
+      <minDepth>0.01</minDepth>
+      <material>Gazebo/DarkGrey</material>
     </gazebo>
   </xacro:macro>
@@ -148,10 +139,12 @@
     </link>
     <gazebo reference="${prefix}${fingerprefix}_inner_finger">
-      <implicitSpringDamper>1</implicitSpringDamper>
-      <mu1>100000</mu1>
-      <mu2>100000</mu2>
-      <kp>100000000.0</kp>
-      <kd>1.0</kd>
-      <material>Gazebo/Black</material>
+      <kp>1000000.0</kp>
+      <kd>100.0</kd>
+      <mu1>1000.0</mu1>
+      <mu2>1000.0</mu2>
+      <fdir1>0 0 0</fdir1>
+      <maxVel>1.0</maxVel>
+      <minDepth>0.01</minDepth>
+      <material>Gazebo/DarkGrey</material>
     </gazebo>
   </xacro:macro>
@@ -179,10 +172,12 @@
     </link>
     <gazebo reference="${prefix}${fingerprefix}_inner_finger_pad">
-      <implicitSpringDamper>1</implicitSpringDamper>
-      <mu1>100000</mu1>
-      <mu2>100000</mu2>
-      <kp>100000000.0</kp>
-      <kd>1.0</kd>
-      <material>Gazebo/DarkGrey</material>
+      <kp>1000000.0</kp>
+      <kd>100.0</kd>
+      <mu1>1000.0</mu1>
+      <mu2>1000.0</mu2>
+      <fdir1>0 0 0</fdir1>
+      <maxVel>1.0</maxVel>
+      <minDepth>0.01</minDepth>
+      <material>Gazebo/LightGrey</material>
     </gazebo>
   </xacro:macro>
@@ -201,5 +196,5 @@
       <child link="${prefix}${fingerprefix}_inner_knuckle" />
       <axis xyz="1 0 0" />
-      <limit lower="-0.8757" upper="0.8757" velocity="2.0" effort="1000" />
+      <limit lower="-0.8757" upper="0.8757" velocity="0.5" effort="0.05" />
       <mimic joint="${prefix}finger_joint" multiplier="-1" offset="0" />
     </joint>
@@ -212,5 +207,5 @@
       <child link="${prefix}${fingerprefix}_inner_finger" />
       <axis xyz="1 0 0" />
-      <limit lower="-0.8757" upper="0.8757" velocity="2.0" effort="1000" />
+      <limit lower="-0.8757" upper="0.8757" velocity="0.5" effort="0.05" />
       <mimic joint="${prefix}finger_joint" multiplier="1" offset="0" />
     </joint>
@@ -249,7 +244,5 @@
     </link>
     <gazebo reference="${prefix}base_link">
-      <mu1>0.9</mu1>
-      <mu2>0.9</mu2>
-      <material>Gazebo/Black</material>
+      <material>Gazebo/DarkGrey</material>
     </gazebo>
   </xacro:macro>
@@ -280,7 +273,5 @@
     </link>
     <gazebo reference="${prefix}coupler_link">
-      <mu1>0.9</mu1>
-      <mu2>0.9</mu2>
-      <material>Gazebo/Black</material>
+      <material>Gazebo/DarkGrey</material>
     </gazebo>
   </xacro:macro>
@@ -318,6 +309,11 @@
       <child link="${prefix}left_outer_knuckle" />
       <axis xyz="-1 0 0" />
-      <limit lower="0" upper="0.7" velocity="2.0" effort="1000" />
-    </joint>
+      <limit lower="0" upper="0.7" velocity="0.5" effort="0.05" />
+      <dynamics damping="0.2"/>
+    </joint>
+    <gazebo reference="${prefix}finger_joint">
+      <implicitSpringDamper>1</implicitSpringDamper>
+      <provideFeedback>1</provideFeedback>
+    </gazebo>
     <xacro:finger_joints prefix="${prefix}" fingerprefix="left" reflect="1.0"/>
   </xacro:macro>
@@ -328,5 +324,5 @@
       <child link="${prefix}right_outer_knuckle" />
       <axis xyz="1 0 0" />
-      <limit lower="-0.725" upper="0.725" velocity="2.0" effort="1000" />
+      <limit lower="-0.725" upper="0.725" velocity="0.5" effort="0.05" />
     <mimic joint="${prefix}finger_joint" multiplier="-1" offset="0" />
     </joint>

File: pal_robotiq_85_gripper/pal_robotiq_85_description/urdf/robotiq_85_gripper.urdf.xacro (robot description, xacro)
@@ -2,7 +2,9 @@
 <robot xmlns:xacro="http://ros.org/wiki/xacro">
   <xacro:include filename="$(find pal_robotiq_85_description)/urdf/robotiq_85_gripper.transmission.xacro" />
-  <xacro:macro name="mimic_joint_plugin_gazebo" params="name_prefix parent_joint mimic_joint has_pid:=false multiplier:=1.0 offset:=0 sensitiveness:=0.0 max_effort:=10.0 robot_namespace:=''">
+  <xacro:property name="finger_joint_damping" value="0.0025"/>
+  <xacro:property name="finger_joint_friction" value="0.0"/>
+  <xacro:macro name="mimic_joint_plugin_gazebo" params="name_prefix parent_joint mimic_joint has_pid:=false multiplier:=1.0 offset:=0 sensitiveness:=0.0 max_effort:=0.05 robot_namespace:=''">
     <gazebo>
-      <plugin name="${name_prefix}mimic_joint_plugin" filename="libroboticsgroup_gazebo_mimic_joint_plugin.so">
+      <plugin name="${name_prefix}mimic_joint_plugin" filename="libroboticsgroup_upatras_gazebo_mimic_joint_plugin.so">
         <joint>${parent_joint}</joint>
         <mimicJoint>${mimic_joint}</mimicJoint>
@@ -23,7 +25,9 @@
     <link name="${prefix}${fingerprefix}_outer_knuckle">
       <inertial>
-        <origin xyz="${reflect * 0.01545} 0 -0.00118" rpy="0 0 0" />
-        <mass value="0.01252" />
-        <inertia ixx="312.44E-9" ixy="0" ixz="-168.09E-9" iyy="2156E-9" iyz="0" izz="2027.51E-9" />
+          <mass value="0.018491" />
+          <origin xyz="0.0 0.0 0.0" />
+          <inertia ixx = "0.000009" ixy = "-0.000001" ixz = "0.000000"
+                   iyx = "-0.000001" iyy = "0.000001" iyz = "0.000000"
+                   izx = "0.000000" izy = "0.000000" izz = "0.000010" />
       </inertial>
       <visual>
@@ -43,19 +47,13 @@
       </collision>
     </link>
-    <gazebo reference="${prefix}${fingerprefix}_outer_knuckle">
-        <implicitSpringDamper>1</implicitSpringDamper>
-        <mu1>100000</mu1>
-        <mu2>100000</mu2>
-        <kp>100000000.0</kp>
-        <kd>1.0</kd>
-        <material>Gazebo/DarkGrey</material>
-    </gazebo>
   </xacro:macro>
   <xacro:macro name="outer_finger" params="prefix fingerprefix reflect">
     <link name="${prefix}${fingerprefix}_outer_finger">
       <inertial>
-        <origin xyz="0.004 0 ${reflect * 0.01892}" rpy="0 0 0" />
-        <mass value="0.03848" />
-        <inertia ixx="12341E-9" ixy="0" ixz="-2152.21E-9" iyy="10617E-9" iyz="0" izz="4812.09E-9" />
+          <mass value="0.027309" />
+          <origin xyz="0.0 0.0 0.0" />
+          <inertia ixx = "0.000003" ixy = "-0.000002" ixz = "0.000000"
+                   iyx = "-0.000002" iyy = "0.000021" iyz = "0.000000"
+                   izx = "0.000000" izy = "0.000000" izz = "0.000020" />
       </inertial>
       <visual>
@@ -75,10 +73,6 @@
       </collision>
     </link>
-    <gazebo reference="{prefix}${fingerprefix}_outer_finger">
-        <implicitSpringDamper>1</implicitSpringDamper>
-        <mu1>100000</mu1>
-        <mu2>100000</mu2>
-        <kp>100000000.0</kp>
-        <kd>1.0</kd>
+    <gazebo reference="${prefix}${fingerprefix}_outer_finger">
+      <material>Gazebo/DarkGrey</material>
     </gazebo>
   </xacro:macro>
@@ -86,7 +80,9 @@
     <link name="${prefix}${fingerprefix}_inner_knuckle">
       <inertial>
-        <origin xyz="${reflect * 0.01952} 0 0.022" rpy="0 0 0" />
-        <mass value="0.02731" />
-        <inertia ixx="8621.3E-9" ixy="0" ixz="-3646.49E-9" iyy="8004.28E-9" iyz="0" izz="7704.42E-9" />
+          <mass value="0.029951" />
+          <origin xyz="0.0 0.0 0.0" />
+          <inertia ixx = "0.000039" ixy = "0.000000" ixz = "0.000000"
+                   iyx = "0.000000" iyy = "0.000005" iyz = "0.000000"
+                   izx = "0.000000" izy = "0.000000" izz = "0.000035" />
       </inertial>
       <visual>
@@ -107,9 +103,12 @@
     </link>
     <gazebo reference="${prefix}${fingerprefix}_inner_knuckle">
-        <implicitSpringDamper>1</implicitSpringDamper>
-        <mu1>100000</mu1>
-        <mu2>100000</mu2>
-        <kp>100000000.0</kp>
-        <kd>1.0</kd>
+      <kp>1000000.0</kp>
+      <kd>100.0</kd>
+      <mu1>1000.0</mu1>
+      <mu2>1000.0</mu2>
+      <fdir1>0 0 0</fdir1>
+      <maxVel>1.0</maxVel>
+      <minDepth>0.01</minDepth>
+      <material>Gazebo/DarkGrey</material>
     </gazebo>
   </xacro:macro>
@@ -117,7 +116,9 @@
     <link name="${prefix}${fingerprefix}_inner_finger">
       <inertial>
-        <origin xyz="${reflect * -0.01409} 0 0.01569" rpy="0 0 0" />
-        <mass value="0.037" />
-        <inertia ixx="12446.57E-9" ixy="0" ixz="4167.81E-9" iyy="14201.18E-9" iyz="0" izz="4979.86E-9" />
+          <mass value="0.019555" />
+          <origin xyz="0.0 0.0 0.0" />
+          <inertia ixx = "0.000002" ixy = "0.000000" ixz = "0.000000"
+                   iyx = "0.000000" iyy = "0.000005" iyz = "0.000000"
+                   izx = "0.000000" izy = "0.000000" izz = "0.000006" />
       </inertial>
       <visual>
@@ -138,9 +139,12 @@
     </link>
     <gazebo reference="${prefix}${fingerprefix}_inner_finger">
-        <implicitSpringDamper>1</implicitSpringDamper>
-        <mu1>100000</mu1>
-        <mu2>100000</mu2>
-        <kp>100000000.0</kp>
-        <kd>1.0</kd>
+      <kp>1000000.0</kp>
+      <kd>100.0</kd>
+      <mu1>1000.0</mu1>
+      <mu2>1000.0</mu2>
+      <fdir1>0 0 0</fdir1>
+      <maxVel>1.0</maxVel>
+      <minDepth>0.01</minDepth>
+      <material>Gazebo/DarkGrey</material>
     </gazebo>
   </xacro:macro>
@@ -166,11 +170,20 @@
         </material>
       </collision>
+      <inertial>
+          <mass value="0.019555" />
+          <origin xyz="0.0 0.0 0.0" />
+          <inertia ixx = "0.000002" ixy = "0.000000" ixz = "0.000000"
+                   iyx = "0.000000" iyy = "0.000005" iyz = "0.000000"
+                   izx = "0.000000" izy = "0.000000" izz = "0.000006" />
+      </inertial>
     </link>
     <gazebo reference="${prefix}${fingerprefix}_inner_finger_pad">
-      <implicitSpringDamper>1</implicitSpringDamper>
-      <mu1>100000</mu1>
-      <mu2>100000</mu2>
-      <kp>100000000.0</kp>
-      <kd>1.0</kd>
+      <kp>1000000.0</kp>
+      <kd>100.0</kd>
+      <mu1>1000.0</mu1>
+      <mu2>1000.0</mu2>
+      <fdir1>0 0 0</fdir1>
+      <maxVel>1.0</maxVel>
+      <minDepth>0.01</minDepth>
       <material>Gazebo/DarkGrey</material>
     </gazebo>
@@ -183,4 +196,8 @@
       <axis xyz="1 0 0" />
     </joint>
+    <gazebo reference="${prefix}${fingerprefix}_outer_finger_joint">
+      <provideFeedback>1</provideFeedback>
+      <implicitSpringDamper>1</implicitSpringDamper>
+    </gazebo>
   </xacro:macro>
   <xacro:macro name="inner_knuckle_joint" params="prefix fingerprefix reflect">
@@ -191,5 +208,5 @@
       <child link="${prefix}${fingerprefix}_inner_knuckle" />
       <axis xyz="1 0 0" />
-      <limit lower="0" upper="0.8757" velocity="2.0" effort="1000" />
+      <limit lower="0" upper="0.8757" velocity="0.5" effort="0.05" />
       <mimic joint="${prefix}finger_joint" multiplier="1" offset="0" />
     </joint>
@@ -202,5 +219,5 @@
       <child link="${prefix}${fingerprefix}_inner_finger" />
       <axis xyz="1 0 0" />
-      <limit lower="-0.8757" upper="0" velocity="2.0" effort="1000" />
+      <limit lower="-0.8757" upper="0" velocity="0.5" effort="0.05" />
       <mimic joint="${prefix}finger_joint" multiplier="-1" offset="0" />
     </joint>
@@ -218,7 +235,9 @@
     <link name="${prefix}base_link">
       <inertial>
-        <origin xyz="8.625E-08 -4.6583E-06 0.03145" rpy="0 0 0" />
-        <mass value="0.22652" />
-        <inertia ixx="0.00020005" ixy="-4.2442E-10" ixz="-2.9069E-10" iyy="0.00017832" iyz="-3.4402E-08" izz="0.00013478" />
+          <mass value="0.636951" />
+          <origin xyz="0.0 0.0 0.0" />
+          <inertia ixx = "0.000380" ixy = "0.000000" ixz = "0.000000"
+                   iyx = "0.000000" iyy = "0.001110" iyz = "0.000000"
+                   izx = "0.000000" izy = "0.000000" izz = "0.001171" />
       </inertial>
       <visual>
@@ -239,7 +258,5 @@
     </link>
     <gazebo reference="${prefix}base_link">
-      <mu1>0.9</mu1>
-      <mu2>0.9</mu2>
-      <material>Gazebo/Black</material>
+      <material>Gazebo/DarkGrey</material>
     </gazebo>
   </xacro:macro>
@@ -270,7 +287,5 @@
     </link>
     <gazebo reference="${prefix}coupler_link">
-      <mu1>0.9</mu1>
-      <mu2>0.9</mu2>
-      <material>Gazebo/Black</material>
+      <material>Gazebo/DarkGrey</material>
     </gazebo>
   </xacro:macro>
@@ -308,6 +323,11 @@
       <child link="${prefix}left_outer_knuckle" />
       <axis xyz="1 0 0" />
-      <limit lower="0" upper="0.8" velocity="2.0" effort="1000" />
-    </joint>
+      <limit lower="0" upper="0.8" velocity="0.5" effort="0.05" />
+      <dynamics damping="0.2"/>
+    </joint>
+    <gazebo reference="${prefix}finger_joint">
+      <implicitSpringDamper>1</implicitSpringDamper>
+      <provideFeedback>1</provideFeedback>
+    </gazebo>
     <xacro:finger_joints prefix="${prefix}" fingerprefix="left" reflect="1.0"/>
   </xacro:macro>
@@ -318,5 +338,5 @@
       <child link="${prefix}right_outer_knuckle" />
       <axis xyz="1 0 0" />
-      <limit lower="0" upper="0.81" velocity="2.0" effort="1000" />
+      <limit lower="0" upper="0.81" velocity="0.5" effort="0.05" />
       <mimic joint="${prefix}finger_joint" multiplier="1" offset="0" />
     </joint>

Commit message: Fix aborted error for robotiq 2f 140

File: pal_robotiq_140_gripper/pal_robotiq_140_description/urdf/robotiq_140_gripper.urdf.xacro (robot description, xacro)
@@ -196,5 +196,5 @@
       <child link="${prefix}${fingerprefix}_inner_knuckle" />
       <axis xyz="1 0 0" />
-      <limit lower="-0.8757" upper="0.8757" velocity="0.5" effort="0.05" />
+      <limit lower="-0.8757" upper="0.8757" velocity="2" effort="0.05" />
       <mimic joint="${prefix}finger_joint" multiplier="-1" offset="0" />
     </joint>
@@ -207,5 +207,5 @@
       <child link="${prefix}${fingerprefix}_inner_finger" />
       <axis xyz="1 0 0" />
-      <limit lower="-0.8757" upper="0.8757" velocity="0.5" effort="0.05" />
+      <limit lower="-0.8757" upper="0.8757" velocity="2" effort="0.05" />
       <mimic joint="${prefix}finger_joint" multiplier="1" offset="0" />
     </joint>
@@ -309,6 +309,6 @@
       <child link="${prefix}left_outer_knuckle" />
       <axis xyz="-1 0 0" />
-      <limit lower="0" upper="0.7" velocity="0.5" effort="0.05" />
-      <dynamics damping="0.2"/>
+      <limit lower="0" upper="0.7" velocity="2" effort="0.05" />
+      <dynamics damping="0.03"/>
     </joint>
     <gazebo reference="${prefix}finger_joint">
@@ -324,5 +324,5 @@
       <child link="${prefix}right_outer_knuckle" />
       <axis xyz="1 0 0" />
-      <limit lower="-0.725" upper="0.725" velocity="0.5" effort="0.05" />
+      <limit lower="-0.725" upper="0.725" velocity="2" effort="0.05" />
     <mimic joint="${prefix}finger_joint" multiplier="-1" offset="0" />
     </joint>

Commit message: Add grasping frame

File: pal_robotiq_140_gripper/pal_robotiq_140_description/urdf/robotiq_140_gripper.urdf.xacro (robot description, xacro)
@@ -276,4 +276,21 @@
     </gazebo>
   </xacro:macro>
+  <!-- Grasping frame -->
+  <xacro:macro name="pal_robotiq_grasping_frame" params="prefix">
+    <joint name="${prefix}grasping_frame_joint" type="fixed">
+      <parent link="${prefix}base_link" />
+      <child link="${prefix}grasping_frame" />
+      <origin xyz="0 0 0.10" rpy="0 -1.5708 0" />
+    </joint>
+    <link name="${prefix}grasping_frame">
+      <inertial>
+        <origin xyz="0 0 0" rpy="0 0 0" />
+        <mass value="0.0001" />
+        <inertia ixx="0.00001" ixy="0.0" ixz="0.0"
+                 iyy="0.00001" iyz="0.0"
+                 izz="0.00001" />
+      </inertial>
+    </link>
+  </xacro:macro>
   <xacro:macro name="pal_robotiq_coupling_joint" params="prefix parent *origin">
     <joint name="${prefix}coupler_joint" type="fixed">
@@ -332,4 +349,5 @@
   <xacro:macro name="robotiq_140_gripper" params="prefix parent *origin">
     <xacro:base_link prefix="${prefix}"/>
+    <xacro:pal_robotiq_grasping_frame prefix="${prefix}"/>
     <xacro:pal_robotiq_coupling_link prefix="${prefix}"/>
     <xacro:finger_links prefix="${prefix}" fingerprefix="left" stroke="140"/>

File: pal_robotiq_85_gripper/pal_robotiq_85_description/urdf/robotiq_85_gripper.urdf.xacro (robot description, xacro)
@@ -286,4 +286,21 @@
     </gazebo>
   </xacro:macro>
+    <!-- Grasping frame -->
+  <xacro:macro name="pal_robotiq_grasping_frame" params="prefix">
+    <joint name="${prefix}grasping_frame_joint" type="fixed">
+      <parent link="${prefix}base_link" />
+      <child link="${prefix}grasping_frame" />
+      <origin xyz="0 0 0.12" rpy="0 -1.5708 0" />
+    </joint>
+    <link name="${prefix}grasping_frame">
+      <inertial>
+        <origin xyz="0 0 0" rpy="0 0 0" />
+        <mass value="0.0001" />
+        <inertia ixx="0.00001" ixy="0.0" ixz="0.0"
+                 iyy="0.00001" iyz="0.0"
+                 izz="0.00001" />
+      </inertial>
+    </link>
+  </xacro:macro>
   <xacro:macro name="pal_robotiq_coupling_joint" params="prefix parent *origin">
     <joint name="${prefix}coupler_joint" type="fixed">
@@ -343,4 +360,5 @@
   <xacro:macro name="robotiq_85_gripper" params="prefix parent *origin">
     <xacro:robotiq_base_link prefix="${prefix}"/>
+    <xacro:pal_robotiq_grasping_frame prefix="${prefix}"/>
     <xacro:pal_robotiq_coupling_link prefix="${prefix}"/>
     <xacro:finger_links prefix="${prefix}" fingerprefix="left" reflect="1"/>
