Commit message: Add fake grasp to 140 + comment the fake grasp

File: pal_robotiq_140_gripper/pal_robotiq_140_description/urdf/robotiq_140_gripper.urdf.xacro (robot description, xacro)
@@ -22,4 +22,19 @@
     </gazebo>
   </xacro:macro>
+  <!-- Add a grasp hack that attach the object when grasped by the gripper to prevent it from falling -->
+  <xacro:macro name="grasp_hack" params="name name_prefix_left name_prefix_right parent_joint">
+    <gazebo>
+      <gripper name="${name}">
+        <grasp_check>
+          <attach_steps>1</attach_steps>
+          <detach_steps>1</detach_steps>
+          <min_contact_count>2</min_contact_count>
+        </grasp_check>
+        <gripper_link>${name_prefix_left}</gripper_link>
+        <gripper_link>${name_prefix_right}</gripper_link>
+        <palm_link>${parent_joint}</palm_link>
+      </gripper>
+    </gazebo>
+  </xacro:macro>
   <xacro:macro name="outer_knuckle" params="prefix fingerprefix stroke">
     <link name="${prefix}${fingerprefix}_outer_knuckle">
@@ -105,8 +120,8 @@
       <kp>1000000.0</kp>
       <kd>100.0</kd>
-      <mu1>1000.0</mu1>
-      <mu2>1000.0</mu2>
+      <mu1>Inf</mu1>
+      <mu2>Inf</mu2>
       <fdir1>0 0 0</fdir1>
-      <maxVel>1.0</maxVel>
+      <maxVel>0.0</maxVel>
       <minDepth>0.01</minDepth>
       <material>Gazebo/DarkGrey</material>
@@ -139,11 +154,28 @@
     </link>
     <gazebo reference="${prefix}${fingerprefix}_inner_finger">
-      <kp>1000000.0</kp>
+      <collision name="${prefix}${fingerprefix}_inner_finger">
+        <surface>
+          <friction>
+            <torsional>
+              <coefficient>1000.0</coefficient>
+              <use_patch_radius>true</use_patch_radius>
+              <patch_radius>0.1</patch_radius>
+            </torsional>
+          </friction>
+          <contact>
+            <poissons_ratio>1.0</poissons_ratio>
+            <elastic_modulus>Inf</elastic_modulus>
+          </contact>
+        </surface>
+      </collision>
+      <mu1>Inf</mu1>
+      <mu2>Inf</mu2>
+      <maxVel>0.0</maxVel>
+      <kp>Inf</kp>
       <kd>100.0</kd>
-      <mu1>1000.0</mu1>
-      <mu2>1000.0</mu2>
-      <fdir1>0 0 0</fdir1>
-      <maxVel>1.0</maxVel>
+      <fdir1>1 0 0</fdir1>
+      <maxVel>0.0</maxVel>
       <minDepth>0.01</minDepth>
+      <maxContacts>100</maxContacts>
       <material>Gazebo/DarkGrey</material>
     </gazebo>
@@ -171,14 +203,4 @@
       </collision>
     </link>
-    <gazebo reference="${prefix}${fingerprefix}_inner_finger_pad">
-      <kp>1000000.0</kp>
-      <kd>100.0</kd>
-      <mu1>1000.0</mu1>
-      <mu2>1000.0</mu2>
-      <fdir1>0 0 0</fdir1>
-      <maxVel>1.0</maxVel>
-      <minDepth>0.01</minDepth>
-      <material>Gazebo/LightGrey</material>
-    </gazebo>
   </xacro:macro>
   <xacro:macro name="outer_finger_joint" params="prefix fingerprefix">
@@ -360,4 +382,5 @@
     <xacro:right_outer_knuckle_joint prefix="${prefix}"/>
     <xacro:robotiq_140_gripper_transmission prefix="${prefix}"/>
+    <!-- <xacro:grasp_hack name="${prefix}grasp_hack" name_prefix_left="${prefix}left_inner_finger" name_prefix_right="${prefix}right_inner_finger" parent_joint="${parent}"/> -->
   </xacro:macro>
 </robot>

File: pal_robotiq_85_gripper/pal_robotiq_85_description/urdf/robotiq_85_gripper.urdf.xacro (robot description, xacro)
@@ -22,4 +22,19 @@
     </gazebo>
   </xacro:macro>
+  <!-- Add a grasp check hack that attach the object to the parent link when grasped by the gripper to prevent it from falling -->
+  <xacro:macro name="grasp_hack" params="name name_prefix_left name_prefix_right parent_joint">
+    <gazebo>
+      <gripper name="${name}_grasp_hack">
+        <grasp_check>
+          <attach_steps>1</attach_steps>
+          <detach_steps>1</detach_steps>
+          <min_contact_count>2</min_contact_count>
+        </grasp_check>
+        <gripper_link>${name_prefix_left}</gripper_link>
+        <gripper_link>${name_prefix_right}</gripper_link>
+        <palm_link>${parent_joint}</palm_link>
+      </gripper>
+    </gazebo>
+  </xacro:macro>
   <xacro:macro name="outer_knuckle" params="prefix fingerprefix reflect">
     <link name="${prefix}${fingerprefix}_outer_knuckle">
@@ -378,16 +393,5 @@
     <xacro:right_outer_knuckle_joint prefix="${prefix}"/>
     <xacro:robotiq_85_gripper_transmission prefix="${prefix}"/>
-  </xacro:macro>
-  <gazebo>
-    <gripper name="${name}_grasp_hack">
-      <grasp_check>
-        <attach_steps>1</attach_steps>
-        <detach_steps>1</detach_steps>
-        <min_contact_count>2</min_contact_count>
-      </grasp_check>
-      <gripper_link>gripper_right_inner_finger</gripper_link>
-      <gripper_link>gripper_left_inner_finger</gripper_link>
-      <palm_link>arm_7_link</palm_link>
-    </gripper>
-  </gazebo>
+    <!-- <xacro:grasp_hack name="${prefix}grasp_hack" name_prefix_left="${prefix}left_inner_finger" name_prefix_right="${prefix}right_inner_finger" parent_joint="${parent}"/> -->
+  </xacro:macro>
 </robot>

Commit message: Update robotiq 140 urdf to increase effort and change grasping frame joint distance

File: pal_robotiq_140_gripper/pal_robotiq_140_description/urdf/robotiq_140_gripper.urdf.xacro (robot description, xacro)
@@ -4,5 +4,5 @@
   <xacro:property name="finger_joint_damping" value="0.0025"/>
   <xacro:property name="finger_joint_friction" value="0.0"/>
-  <xacro:macro name="mimic_joint_plugin_gazebo" params="name_prefix parent_joint mimic_joint has_pid:=false multiplier:=1.0 offset:=0 sensitiveness:=0.0 max_effort:=0.05 robot_namespace:=''">
+  <xacro:macro name="mimic_joint_plugin_gazebo" params="name_prefix parent_joint mimic_joint has_pid:=false multiplier:=1.0 offset:=0 sensitiveness:=0.0 max_effort:=0.12 robot_namespace:=''">
     <gazebo>
       <plugin name="${name_prefix}mimic_joint_plugin" filename="libroboticsgroup_upatras_gazebo_mimic_joint_plugin.so">
@@ -218,5 +218,5 @@
       <child link="${prefix}${fingerprefix}_inner_knuckle" />
       <axis xyz="1 0 0" />
-      <limit lower="-0.8757" upper="0.8757" velocity="2" effort="0.05" />
+      <limit lower="-0.8757" upper="0.8757" velocity="2" effort="0.12" />
       <mimic joint="${prefix}finger_joint" multiplier="-1" offset="0" />
     </joint>
@@ -229,5 +229,5 @@
       <child link="${prefix}${fingerprefix}_inner_finger" />
       <axis xyz="1 0 0" />
-      <limit lower="-0.8757" upper="0.8757" velocity="2" effort="0.05" />
+      <limit lower="-0.8757" upper="0.8757" velocity="2" effort="0.12" />
       <mimic joint="${prefix}finger_joint" multiplier="1" offset="0" />
     </joint>
@@ -303,5 +303,5 @@
       <parent link="${prefix}base_link" />
       <child link="${prefix}grasping_frame" />
-      <origin xyz="0 0 0.10" rpy="0 -1.5708 0" />
+      <origin xyz="0 0 0.14" rpy="0 -1.5708 0" />
     </joint>
     <link name="${prefix}grasping_frame">
@@ -348,5 +348,5 @@
       <child link="${prefix}left_outer_knuckle" />
       <axis xyz="-1 0 0" />
-      <limit lower="0" upper="0.7" velocity="2" effort="0.05" />
+      <limit lower="0" upper="0.7" velocity="2" effort="0.12" />
       <dynamics damping="0.03"/>
     </joint>
@@ -363,5 +363,5 @@
       <child link="${prefix}right_outer_knuckle" />
       <axis xyz="1 0 0" />
-      <limit lower="-0.725" upper="0.725" velocity="2" effort="0.05" />
+      <limit lower="-0.725" upper="0.725" velocity="2" effort="0.12" />
     <mimic joint="${prefix}finger_joint" multiplier="-1" offset="0" />
     </joint>

Commit message: Apply suggestion for naming and syntax

File: pal_robotiq_140_gripper/pal_robotiq_140_description/urdf/robotiq_140_gripper.urdf.xacro (robot description, xacro)
@@ -23,5 +23,5 @@
   </xacro:macro>
   <!-- Add a grasp hack that attach the object when grasped by the gripper to prevent it from falling -->
-  <xacro:macro name="grasp_hack" params="name name_prefix_left name_prefix_right parent_joint">
+  <xacro:macro name="gazebo_gripper_grasp" params="name name_prefix_left name_prefix_right parent_joint">
     <gazebo>
       <gripper name="${name}">
@@ -382,5 +382,5 @@
     <xacro:right_outer_knuckle_joint prefix="${prefix}"/>
     <xacro:robotiq_140_gripper_transmission prefix="${prefix}"/>
-    <xacro:grasp_hack name="${prefix}grasp_hack" name_prefix_left="${prefix}left_inner_finger" name_prefix_right="${prefix}right_inner_finger" parent_joint="${parent}"/>
+    <xacro:gazebo_gripper_grasp name="${prefix}grasp" name_prefix_left="${prefix}left_inner_finger" name_prefix_right="${prefix}right_inner_finger" parent_joint="${parent}"/>
   </xacro:macro>
 </robot>

File: pal_robotiq_85_gripper/pal_robotiq_85_description/urdf/robotiq_85_gripper.urdf.xacro (robot description, xacro)
@@ -22,8 +22,7 @@
     </gazebo>
   </xacro:macro>
-  <!-- Add a grasp check hack that attach the object to the parent link when grasped by the gripper to prevent it from falling -->
-  <xacro:macro name="grasp_hack" params="name name_prefix_left name_prefix_right parent_joint">
+  <xacro:macro name="gazebo_gripper_grasp" params="name name_prefix_left name_prefix_right parent_joint">
     <gazebo>
-      <gripper name="${name}_grasp_hack">
+      <gripper name="${name}">
         <grasp_check>
           <attach_steps>3</attach_steps>    <!-- should not be set to 1 because can cause segfault-->
@@ -393,5 +392,5 @@
     <xacro:right_outer_knuckle_joint prefix="${prefix}"/>
     <xacro:robotiq_85_gripper_transmission prefix="${prefix}"/>
-    <xacro:grasp_hack name="${prefix}grasp_hack" name_prefix_left="${prefix}left_inner_finger" name_prefix_right="${prefix}right_inner_finger" parent_joint="${parent}"/>
+    <xacro:gazebo_gripper_grasp name="${prefix}grasp" name_prefix_left="${prefix}left_inner_finger" name_prefix_right="${prefix}right_inner_finger" parent_joint="${parent}"/>
   </xacro:macro>
 </robot>

Commit message: Added Z and Y grasping frames

File: pal_robotiq_140_gripper/pal_robotiq_140_description/urdf/robotiq_140_gripper.urdf.xacro (robot description, xacro)
@@ -315,4 +315,38 @@
     </link>
   </xacro:macro>
+  <!-- Grasping frame Y -->
+  <xacro:macro name="pal_robotiq_grasping_frame_Y" params="prefix">
+    <joint name="${prefix}grasping_frame_Y_joint" type="fixed">
+      <parent link="${prefix}base_link" />
+      <child link="${prefix}grasping_frame_Y" />
+      <origin xyz="0 0 0.14" rpy="1.5708 0 -3.1416" />
+    </joint>
+    <link name="${prefix}grasping_frame_Y">
+      <inertial>
+        <origin xyz="0 0 0" rpy="0 0 0" />
+        <mass value="0.0001" />
+        <inertia ixx="0.00001" ixy="0.0" ixz="0.0"
+                 iyy="0.00001" iyz="0.0"
+                 izz="0.00001" />
+      </inertial>
+    </link>
+  </xacro:macro>
+    <!-- Grasping frame Z -->
+  <xacro:macro name="pal_robotiq_grasping_frame_Z" params="prefix">
+    <joint name="${prefix}grasping_frame_Z_joint" type="fixed">
+      <parent link="${prefix}base_link" />
+      <child link="${prefix}grasping_frame_Z" />
+      <origin xyz="0 0 0.14" rpy="0 0 3.1416" />
+    </joint>
+    <link name="${prefix}grasping_frame_Z">
+      <inertial>
+        <origin xyz="0 0 0" rpy="0 0 0" />
+        <mass value="0.0001" />
+        <inertia ixx="0.00001" ixy="0.0" ixz="0.0"
+                 iyy="0.00001" iyz="0.0"
+                 izz="0.00001" />
+      </inertial>
+    </link>
+  </xacro:macro>
   <xacro:macro name="pal_robotiq_coupling_joint" params="prefix parent *origin">
     <joint name="${prefix}coupler_joint" type="fixed">
@@ -372,4 +406,6 @@
     <xacro:base_link prefix="${prefix}"/>
     <xacro:pal_robotiq_grasping_frame prefix="${prefix}"/>
+    <xacro:pal_robotiq_grasping_frame_Y prefix="${prefix}"/>
+    <xacro:pal_robotiq_grasping_frame_Z prefix="${prefix}"/>
     <xacro:pal_robotiq_coupling_link prefix="${prefix}"/>
     <xacro:finger_links prefix="${prefix}" fingerprefix="left" stroke="140"/>

File: pal_robotiq_85_gripper/pal_robotiq_85_description/urdf/robotiq_85_gripper.urdf.xacro (robot description, xacro)
@@ -312,7 +312,41 @@
       <parent link="${prefix}base_link" />
       <child link="${prefix}grasping_frame" />
-      <origin xyz="0 0 0.10" rpy="0 -1.5708 0" />
+      <origin xyz="0 0 0.11" rpy="0 -1.5708 0" />
     </joint>
     <link name="${prefix}grasping_frame">
+      <inertial>
+        <origin xyz="0 0 0" rpy="0 0 0" />
+        <mass value="0.0001" />
+        <inertia ixx="0.00001" ixy="0.0" ixz="0.0"
+                 iyy="0.00001" iyz="0.0"
+                 izz="0.00001" />
+      </inertial>
+    </link>
+  </xacro:macro>
+  <!-- Grasping frame Y -->
+  <xacro:macro name="pal_robotiq_grasping_frame_Y" params="prefix">
+    <joint name="${prefix}grasping_frame_Y_joint" type="fixed">
+      <parent link="${prefix}base_link" />
+      <child link="${prefix}grasping_frame_Y" />
+      <origin xyz="0 0 0.11" rpy="1.5708 0 -3.1416" />
+    </joint>
+    <link name="${prefix}grasping_frame_Y">
+      <inertial>
+        <origin xyz="0 0 0" rpy="0 0 0" />
+        <mass value="0.0001" />
+        <inertia ixx="0.00001" ixy="0.0" ixz="0.0"
+                 iyy="0.00001" iyz="0.0"
+                 izz="0.00001" />
+      </inertial>
+    </link>
+  </xacro:macro>
+    <!-- Grasping frame Z -->
+  <xacro:macro name="pal_robotiq_grasping_frame_Z" params="prefix">
+    <joint name="${prefix}grasping_frame_Z_joint" type="fixed">
+      <parent link="${prefix}base_link" />
+      <child link="${prefix}grasping_frame_Z" />
+      <origin xyz="0 0 0.11" rpy="0 0 0" />
+    </joint>
+    <link name="${prefix}grasping_frame_Z">
       <inertial>
         <origin xyz="0 0 0" rpy="0 0 0" />
@@ -382,4 +416,6 @@
     <xacro:robotiq_base_link prefix="${prefix}"/>
     <xacro:pal_robotiq_grasping_frame prefix="${prefix}"/>
+    <xacro:pal_robotiq_grasping_frame_Y prefix="${prefix}"/>
+    <xacro:pal_robotiq_grasping_frame_Z prefix="${prefix}"/>
     <xacro:pal_robotiq_coupling_link prefix="${prefix}"/>
     <xacro:finger_links prefix="${prefix}" fingerprefix="left" reflect="1"/>

File: pal_robotiq_epick_gripper/pal_robotiq_epick_description/urdf/robotiq_epick_model_macro.xacro (robot description, xacro)
@@ -120,4 +120,34 @@
       </inertial>
     </link>
+    <!-- Graping Frame Y -->
+    <joint name="${prefix}grasping_frame_Y_joint" type="fixed">
+      <parent link="${prefix}base_link" />
+      <child link="${prefix}grasping_frame_Y" />
+      <origin xyz="0 0 0.135" rpy="1.5708 0 -3.1416" />
+    </joint>
+    <link name="${prefix}grasping_frame_Y">
+      <inertial>
+        <origin xyz="0 0 0" rpy="0 0 0" />
+        <mass value="0.0001" />
+        <inertia ixx="0.00001" ixy="0.0" ixz="0.0"
+                iyy="0.00001" iyz="0.0"
+                izz="0.00001" />
+      </inertial>
+    </link>
+    <!-- Graping Frame Z -->
+    <joint name="${prefix}grasping_frame_Z_joint" type="fixed">
+      <parent link="${prefix}base_link" />
+      <child link="${prefix}grasping_frame_Z" />
+      <origin xyz="0 0 0.135" rpy="0 0 3.1416" />
+    </joint>
+    <link name="${prefix}grasping_frame_Z">
+      <inertial>
+        <origin xyz="0 0 0" rpy="0 0 0" />
+        <mass value="0.0001" />
+        <inertia ixx="0.00001" ixy="0.0" ixz="0.0"
+                iyy="0.00001" iyz="0.0"
+                izz="0.00001" />
+      </inertial>
+    </link>
     <xacro:robotiq_epick_gripper_transmission prefix="${prefix}"/>
   </xacro:macro>
