Commit message: Replaced links by grasping frames macro

File: pal_robotiq_140_gripper/pal_robotiq_140_description/urdf/robotiq_140_gripper.urdf.xacro (robot description, xacro)
@@ -2,4 +2,5 @@
 <robot xmlns:xacro="http://ros.org/wiki/xacro">
   <xacro:include filename="$(find pal_robotiq_140_description)/urdf/robotiq_140_gripper.transmission.xacro" />
+  <xacro:include filename="$(find tiago_description)/urdf/end_effector/grasping_frames.xacro" />
   <xacro:property name="finger_joint_damping" value="0.0025"/>
   <xacro:property name="finger_joint_friction" value="0.0"/>
@@ -298,55 +299,4 @@
     </gazebo>
   </xacro:macro>
-  <!-- Grasping frame -->
-  <xacro:macro name="pal_robotiq_grasping_frame" params="prefix">
-    <joint name="${prefix}grasping_frame_joint" type="fixed">
-      <parent link="${prefix}base_link" />
-      <child link="${prefix}grasping_frame" />
-      <origin xyz="0 0 0.14" rpy="0 -1.5708 0" />
-    </joint>
-    <link name="${prefix}grasping_frame">
-      <inertial>
-        <origin xyz="0 0 0" rpy="0 0 0" />
-        <mass value="0.0001" />
-        <inertia ixx="0.00001" ixy="0.0" ixz="0.0"
-                 iyy="0.00001" iyz="0.0"
-                 izz="0.00001" />
-      </inertial>
-    </link>
-  </xacro:macro>
-  <!-- Grasping frame Y -->
-  <xacro:macro name="pal_robotiq_grasping_frame_Y" params="prefix">
-    <joint name="${prefix}grasping_frame_Y_joint" type="fixed">
-      <parent link="${prefix}base_link" />
-      <child link="${prefix}grasping_frame_Y" />
-      <origin xyz="0 0 0.14" rpy="1.5708 0 -3.1416" />
-    </joint>
-    <link name="${prefix}grasping_frame_Y">
-      <inertial>
-        <origin xyz="0 0 0" rpy="0 0 0" />
-        <mass value="0.0001" />
-        <inertia ixx="0.00001" ixy="0.0" ixz="0.0"
-                 iyy="0.00001" iyz="0.0"
-                 izz="0.00001" />
-      </inertial>
-    </link>
-  </xacro:macro>
-    <!-- Grasping frame Z -->
-  <xacro:macro name="pal_robotiq_grasping_frame_Z" params="prefix">
-    <joint name="${prefix}grasping_frame_Z_joint" type="fixed">
-      <parent link="${prefix}base_link" />
-      <child link="${prefix}grasping_frame_Z" />
-      <origin xyz="0 0 0.14" rpy="0 0 3.1416" />
-    </joint>
-    <link name="${prefix}grasping_frame_Z">
-      <inertial>
-        <origin xyz="0 0 0" rpy="0 0 0" />
-        <mass value="0.0001" />
-        <inertia ixx="0.00001" ixy="0.0" ixz="0.0"
-                 iyy="0.00001" iyz="0.0"
-                 izz="0.00001" />
-      </inertial>
-    </link>
-  </xacro:macro>
   <xacro:macro name="pal_robotiq_coupling_joint" params="prefix parent *origin">
     <joint name="${prefix}coupler_joint" type="fixed">
@@ -405,7 +355,5 @@
   <xacro:macro name="robotiq_140_gripper" params="prefix parent *origin">
     <xacro:base_link prefix="${prefix}"/>
-    <xacro:pal_robotiq_grasping_frame prefix="${prefix}"/>
-    <xacro:pal_robotiq_grasping_frame_Y prefix="${prefix}"/>
-    <xacro:pal_robotiq_grasping_frame_Z prefix="${prefix}"/>
+    <xacro:pal_robotiq_grasping_frames prefix="${prefix}" xyz="0 0 0.14"/>
     <xacro:pal_robotiq_coupling_link prefix="${prefix}"/>
     <xacro:finger_links prefix="${prefix}" fingerprefix="left" stroke="140"/>

File: pal_robotiq_85_gripper/pal_robotiq_85_description/urdf/robotiq_85_gripper.urdf.xacro (robot description, xacro)
@@ -2,4 +2,5 @@
 <robot xmlns:xacro="http://ros.org/wiki/xacro">
   <xacro:include filename="$(find pal_robotiq_85_description)/urdf/robotiq_85_gripper.transmission.xacro" />
+  <xacro:include filename="$(find tiago_description)/urdf/end_effector/grasping_frames.xacro" />
   <xacro:property name="finger_joint_damping" value="0.0025"/>
   <xacro:property name="finger_joint_friction" value="0.0"/>
@@ -307,55 +308,4 @@
     </gazebo>
   </xacro:macro>
-    <!-- Grasping frame -->
-  <xacro:macro name="pal_robotiq_grasping_frame" params="prefix">
-    <joint name="${prefix}grasping_frame_joint" type="fixed">
-      <parent link="${prefix}base_link" />
-      <child link="${prefix}grasping_frame" />
-      <origin xyz="0 0 0.11" rpy="0 -1.5708 0" />
-    </joint>
-    <link name="${prefix}grasping_frame">
-      <inertial>
-        <origin xyz="0 0 0" rpy="0 0 0" />
-        <mass value="0.0001" />
-        <inertia ixx="0.00001" ixy="0.0" ixz="0.0"
-                 iyy="0.00001" iyz="0.0"
-                 izz="0.00001" />
-      </inertial>
-    </link>
-  </xacro:macro>
-  <!-- Grasping frame Y -->
-  <xacro:macro name="pal_robotiq_grasping_frame_Y" params="prefix">
-    <joint name="${prefix}grasping_frame_Y_joint" type="fixed">
-      <parent link="${prefix}base_link" />
-      <child link="${prefix}grasping_frame_Y" />
-      <origin xyz="0 0 0.11" rpy="1.5708 0 -3.1416" />
-    </joint>
-    <link name="${prefix}grasping_frame_Y">
-      <inertial>
-        <origin xyz="0 0 0" rpy="0 0 0" />
-        <mass value="0.0001" />
-        <inertia ixx="0.00001" ixy="0.0" ixz="0.0"
-                 iyy="0.00001" iyz="0.0"
-                 izz="0.00001" />
-      </inertial>
-    </link>
-  </xacro:macro>
-    <!-- Grasping frame Z -->
-  <xacro:macro name="pal_robotiq_grasping_frame_Z" params="prefix">
-    <joint name="${prefix}grasping_frame_Z_joint" type="fixed">
-      <parent link="${prefix}base_link" />
-      <child link="${prefix}grasping_frame_Z" />
-      <origin xyz="0 0 0.11" rpy="0 0 0" />
-    </joint>
-    <link name="${prefix}grasping_frame_Z">
-      <inertial>
-        <origin xyz="0 0 0" rpy="0 0 0" />
-        <mass value="0.0001" />
-        <inertia ixx="0.00001" ixy="0.0" ixz="0.0"
-                 iyy="0.00001" iyz="0.0"
-                 izz="0.00001" />
-      </inertial>
-    </link>
-  </xacro:macro>
   <xacro:macro name="pal_robotiq_coupling_joint" params="prefix parent *origin">
     <joint name="${prefix}coupler_joint" type="fixed">
@@ -415,7 +365,5 @@
   <xacro:macro name="robotiq_85_gripper" params="prefix parent *origin">
     <xacro:robotiq_base_link prefix="${prefix}"/>
-    <xacro:pal_robotiq_grasping_frame prefix="${prefix}"/>
-    <xacro:pal_robotiq_grasping_frame_Y prefix="${prefix}"/>
-    <xacro:pal_robotiq_grasping_frame_Z prefix="${prefix}"/>
+    <xacro:pal_robotiq_grasping_frames prefix="${prefix}" xyz="0 0 0.11"/>
     <xacro:pal_robotiq_coupling_link prefix="${prefix}"/>
     <xacro:finger_links prefix="${prefix}" fingerprefix="left" reflect="1"/>

File: pal_robotiq_epick_gripper/pal_robotiq_epick_description/urdf/robotiq_epick_model_macro.xacro (robot description, xacro)
@@ -2,4 +2,5 @@
 <robot xmlns:xacro="http://www.ros.org/wiki/xacro">
   <xacro:include filename="$(find pal_robotiq_epick_description)/urdf/robotiq_epick_gripper.transmission.xacro" />
+  <xacro:include filename="$(find tiago_description)/urdf/end_effector/grasping_frames.xacro" />
   <xacro:property name="joint_lower_limit" value="0.0" />
   <xacro:property name="joint_upper_limit" value="0.055" />
@@ -105,49 +106,5 @@
       </inertial>
     </link>
-    <!-- Graping Frame -->
-    <joint name="${prefix}grasping_frame_joint" type="fixed">
-      <parent link="${prefix}base_link" />
-      <child link="${prefix}grasping_frame" />
-      <origin xyz="0 0 0.135" rpy="0 -1.5708 0" />
-    </joint>
-    <link name="${prefix}grasping_frame">
-      <inertial>
-        <origin xyz="0 0 0" rpy="0 0 0" />
-        <mass value="0.0001" />
-        <inertia ixx="0.00001" ixy="0.0" ixz="0.0"
-                iyy="0.00001" iyz="0.0"
-                izz="0.00001" />
-      </inertial>
-    </link>
-    <!-- Graping Frame Y -->
-    <joint name="${prefix}grasping_frame_Y_joint" type="fixed">
-      <parent link="${prefix}base_link" />
-      <child link="${prefix}grasping_frame_Y" />
-      <origin xyz="0 0 0.135" rpy="1.5708 0 -3.1416" />
-    </joint>
-    <link name="${prefix}grasping_frame_Y">
-      <inertial>
-        <origin xyz="0 0 0" rpy="0 0 0" />
-        <mass value="0.0001" />
-        <inertia ixx="0.00001" ixy="0.0" ixz="0.0"
-                iyy="0.00001" iyz="0.0"
-                izz="0.00001" />
-      </inertial>
-    </link>
-    <!-- Graping Frame Z -->
-    <joint name="${prefix}grasping_frame_Z_joint" type="fixed">
-      <parent link="${prefix}base_link" />
-      <child link="${prefix}grasping_frame_Z" />
-      <origin xyz="0 0 0.135" rpy="0 0 3.1416" />
-    </joint>
-    <link name="${prefix}grasping_frame_Z">
-      <inertial>
-        <origin xyz="0 0 0" rpy="0 0 0" />
-        <mass value="0.0001" />
-        <inertia ixx="0.00001" ixy="0.0" ixz="0.0"
-                iyy="0.00001" iyz="0.0"
-                izz="0.00001" />
-      </inertial>
-    </link>
+    <xacro:pal_robotiq_grasping_frames prefix="${prefix}" xyz="0 0 0.135"/>
     <xacro:robotiq_epick_gripper_transmission prefix="${prefix}"/>
   </xacro:macro>
