Commit message: deleting transmition from the grippers urdfs

File: pal_robotiq_description/urdf/robotiq.transmission.xacro (robot description, xacro)
@@ -13,5 +13,5 @@
  -->
 <robot xmlns:xacro="http://ros.org/wiki/xacro">
-  <xacro:macro name="robotiq_transmission" params="prefix reduction:=1.0">
+  <xacro:macro name="robotiq_transmission" params="prefix reduction">
     <transmission name="${prefix}_trans">
       <plugin>transmission_interface/SimpleTransmission</plugin>

File: pal_robotiq_description/urdf/robotiq_140_gripper.urdf.xacro (robot description, xacro)
@@ -344,5 +344,4 @@
     <xacro:finger_joint prefix="${prefix}"/>
     <xacro:right_outer_knuckle_joint prefix="${prefix}"/>
-    <xacro:robotiq_transmission prefix="${prefix}"/>
     <!--This xacro is used to be able to grasp object in simulmation more robustly, it could cause segfault at grasping time -->
     <xacro:gazebo_gripper_grasp name="${prefix}grasp" name_prefix_left="${prefix}left_inner_finger" name_prefix_right="${prefix}right_inner_finger" parent_joint="${parent}"/>

File: pal_robotiq_description/urdf/robotiq_85_gripper.urdf.xacro (robot description, xacro)
@@ -357,5 +357,4 @@
     <xacro:finger_joint prefix="${prefix}"/>
     <xacro:right_outer_knuckle_joint prefix="${prefix}"/>
-    <xacro:robotiq_transmission prefix="${prefix}"/>
     <!--This xacro is used to be able to grasp object in simulmation more robustly, it could cause segfault at grasping time -->
     <xacro:gazebo_gripper_grasp name="${prefix}grasp" name_prefix_left="${prefix}left_inner_finger" name_prefix_right="${prefix}right_inner_finger" parent_joint="${parent}"/>
