Commit message: adding mimic joints by hand, as result of no library for mimic gazebo

File: pal_robotiq_description/urdf/robotiq.ros2_control.xacro (robot description, xacro)
@@ -13,6 +13,6 @@
  -->
 <robot xmlns:xacro="http://ros.org/wiki/xacro">
-  <xacro:macro name="ros2_control_robotiq_gripper" params="name reduction" >
-    <joint name="${name}_joint">
+  <xacro:macro name="ros2_control_robotiq_85_gripper" params="name reduction" >
+    <joint name="${name}_finger_joint">
       <command_interface name="position" />
       <state_interface name="position" />
@@ -20,6 +20,112 @@
       <state_interface name="effort" />
     </joint>
+    <joint name="${name}_right_outer_knuckle_joint">
+      <param name="mimic">${name}_finger_joint</param>
+      <param name="multiplier">1</param>
+      <command_interface name="position"/>
+      <state_interface name="position"/>
+      <state_interface name="velocity"/>
+      <state_interface name="effort"/>
+    </joint>
+    <joint name="${name}_right_inner_knuckle_joint">
+      <param name="mimic">${name}_finger_joint</param>
+      <param name="multiplier">1</param>
+      <command_interface name="position"/>
+      <state_interface name="position"/>
+      <state_interface name="velocity"/>
+      <state_interface name="effort"/>
+    </joint>
+    <joint name="${name}_right_inner_finger_joint">
+      <param name="mimic">${name}_finger_joint</param>
+      <param name="multiplier">-1</param>
+      <command_interface name="position"/>
+      <state_interface name="position"/>
+      <state_interface name="velocity"/>
+      <state_interface name="effort"/>
+    </joint>
+    <joint name="${name}_left_inner_finger_joint">
+      <param name="mimic">${name}_finger_joint</param>
+      <param name="multiplier">-1</param>
+      <command_interface name="position"/>
+      <state_interface name="position"/>
+      <state_interface name="velocity"/>
+      <state_interface name="effort"/>
+    </joint>
+    <joint name="${name}_left_inner_knuckle_joint">
+      <param name="mimic">${name}_finger_joint</param>
+      <param name="multiplier">1</param>
+      <command_interface name="position"/>
+      <state_interface name="position"/>
+      <state_interface name="velocity"/>
+      <state_interface name="effort"/>
+    </joint>
+    <joint name="${name}_left_outer_knuckle_joint">
+      <param name="mimic">${name}_finger_joint</param>
+      <param name="multiplier">1</param>
+      <command_interface name="position"/>
+      <state_interface name="position"/>
+      <state_interface name="velocity"/>
+      <state_interface name="effort"/>
+    </joint>
     <xacro:include filename="$(find pal_robotiq_description)/urdf/robotiq.transmission.xacro" />
-    <xacro:robotiq_transmission prefix="${name}" reduction="${reduction}" />
+    <xacro:robotiq_transmission prefix="${name}_finger" reduction="${reduction}" />
+  </xacro:macro>
+  <xacro:macro name="ros2_control_robotiq_140_gripper" params="name reduction" >
+    <joint name="${name}_finger_joint">
+      <command_interface name="position" />
+      <state_interface name="position" />
+      <state_interface name="velocity" />
+      <state_interface name="effort" />
+    </joint>
+    <joint name="${name}_right_outer_knuckle_joint">
+      <param name="mimic">${name}_finger_joint</param>
+      <param name="multiplier">-1</param>
+      <command_interface name="position"/>
+      <state_interface name="position"/>
+      <state_interface name="velocity"/>
+      <state_interface name="effort"/>
+    </joint>
+    <joint name="${name}_right_inner_knuckle_joint">
+      <param name="mimic">${name}_finger_joint</param>
+      <param name="multiplier">-1</param>
+      <command_interface name="position"/>
+      <state_interface name="position"/>
+      <state_interface name="velocity"/>
+      <state_interface name="effort"/>
+    </joint>
+    <joint name="${name}_right_inner_finger_joint">
+      <param name="mimic">${name}_finger_joint</param>
+      <param name="multiplier">1</param>
+      <command_interface name="position"/>
+      <state_interface name="position"/>
+      <state_interface name="velocity"/>
+      <state_interface name="effort"/>
+    </joint>
+    <joint name="${name}_left_inner_finger_joint">
+      <param name="mimic">${name}_finger_joint</param>
+      <param name="multiplier">1</param>
+      <command_interface name="position"/>
+      <state_interface name="position"/>
+      <state_interface name="velocity"/>
+      <state_interface name="effort"/>
+    </joint>
+    <joint name="${name}_left_inner_knuckle_joint">
+      <param name="mimic">${name}_finger_joint</param>
+      <param name="multiplier">-1</param>
+      <command_interface name="position"/>
+      <state_interface name="position"/>
+      <state_interface name="velocity"/>
+      <state_interface name="effort"/>
+    </joint>
+    <joint name="${name}_left_outer_knuckle_joint">
+      <param name="mimic">${name}_finger_joint</param>
+      <param name="multiplier">1</param>
+      <command_interface name="position"/>
+      <state_interface name="position"/>
+      <state_interface name="velocity"/>
+      <state_interface name="effort"/>
+    </joint>
+    <xacro:include filename="$(find pal_robotiq_description)/urdf/robotiq.transmission.xacro" />
+    <xacro:robotiq_transmission prefix="${name}_finger" reduction="${reduction}" />
   </xacro:macro>
   <!-- <xacro:macro name="ros2_control_robotiq_epick" params="name reduction" >

Commit message: fix robot description urdf error

File: pal_robotiq_description/urdf/robotiq.ros2_control.xacro (robot description, xacro)
@@ -129,13 +129,3 @@
     <xacro:robotiq_transmission prefix="${name}_finger" reduction="${reduction}" />
   </xacro:macro>
-  <!-- <xacro:macro name="ros2_control_robotiq_epick" params="name reduction" >
-    <joint name="${name}_joint">
-      <command_interface name="effort" />
-      <state_interface name="position" />
-      <state_interface name="velocity" />
-      <state_interface name="effort" />
-    </joint>
-    <xacro:include filename="$(find pal_robotiq_description)/urdf/robotiq.transmission.xacro" />
-    <xacro:robotiq_transmission name="${name}" reduction="${reduction}" />
-  </xacro:macro> -->
 </robot>

Commit message: Add temporary fix for mimic-joint issue https://github.com/ros-controls/gazebo_ros2_control/issues/173

File: pal_robotiq_description/urdf/robotiq.ros2_control.xacro (robot description, xacro)
@@ -13,4 +13,14 @@
  -->
 <robot xmlns:xacro="http://ros.org/wiki/xacro">
+    <xacro:macro name="ros2_control_mimic_joint" params="mimic_joint_name actuated_joint_name multiplier" >
+      <joint name="${mimic_joint_name}">
+        <param name="mimic">${actuated_joint_name}</param>
+        <param name="multiplier">${multiplier}</param>
+        <command_interface name="position" />
+        <state_interface name="position" />
+        <state_interface name="velocity" />
+        <state_interface name="effort" />
+      </joint>
+    </xacro:macro>
   <xacro:macro name="ros2_control_robotiq_85_gripper" params="name reduction" >
     <joint name="${name}_finger_joint">
@@ -20,52 +30,22 @@
       <state_interface name="effort" />
     </joint>
-    <joint name="${name}_right_outer_knuckle_joint">
-      <param name="mimic">${name}_finger_joint</param>
-      <param name="multiplier">1</param>
-      <command_interface name="position"/>
-      <state_interface name="position"/>
-      <state_interface name="velocity"/>
-      <state_interface name="effort"/>
-    </joint>
-    <joint name="${name}_right_inner_knuckle_joint">
-      <param name="mimic">${name}_finger_joint</param>
-      <param name="multiplier">1</param>
-      <command_interface name="position"/>
-      <state_interface name="position"/>
-      <state_interface name="velocity"/>
-      <state_interface name="effort"/>
-    </joint>
-    <joint name="${name}_right_inner_finger_joint">
-      <param name="mimic">${name}_finger_joint</param>
-      <param name="multiplier">-1</param>
-      <command_interface name="position"/>
-      <state_interface name="position"/>
-      <state_interface name="velocity"/>
-      <state_interface name="effort"/>
-    </joint>
-    <joint name="${name}_left_inner_finger_joint">
-      <param name="mimic">${name}_finger_joint</param>
-      <param name="multiplier">-1</param>
-      <command_interface name="position"/>
-      <state_interface name="position"/>
-      <state_interface name="velocity"/>
-      <state_interface name="effort"/>
-    </joint>
-    <joint name="${name}_left_inner_knuckle_joint">
-      <param name="mimic">${name}_finger_joint</param>
-      <param name="multiplier">1</param>
-      <command_interface name="position"/>
-      <state_interface name="position"/>
-      <state_interface name="velocity"/>
-      <state_interface name="effort"/>
-    </joint>
-    <joint name="${name}_left_outer_knuckle_joint">
-      <param name="mimic">${name}_finger_joint</param>
-      <param name="multiplier">1</param>
-      <command_interface name="position"/>
-      <state_interface name="position"/>
-      <state_interface name="velocity"/>
-      <state_interface name="effort"/>
-    </joint>
+    <xacro:ros2_control_mimic_joint mimic_joint_name="${name}_right_outer_knuckle_joint"
+                                    actuated_joint_name="${name}_finger_joint"
+                                    multiplier="1"/>
+   <xacro:ros2_control_mimic_joint mimic_joint_name="${name}_right_inner_knuckle_joint"
+                                    actuated_joint_name="${name}_finger_joint"
+                                    multiplier="1"/>
+    <xacro:ros2_control_mimic_joint mimic_joint_name="${name}_right_inner_finger_joint"
+                                    actuated_joint_name="${name}_finger_joint"
+                                    multiplier="-1"/>
+    <xacro:ros2_control_mimic_joint mimic_joint_name="${name}_left_inner_finger_joint"
+                                    actuated_joint_name="${name}_finger_joint"
+                                    multiplier="-1"/>
+    <xacro:ros2_control_mimic_joint mimic_joint_name="${name}_left_inner_knuckle_joint"
+                                    actuated_joint_name="${name}_finger_joint"
+                                    multiplier="1"/>
+    <xacro:ros2_control_mimic_joint mimic_joint_name="${name}_left_outer_knuckle_joint"
+                                    actuated_joint_name="${name}_finger_joint"
+                                    multiplier="1"/>
     <xacro:include filename="$(find pal_robotiq_description)/urdf/robotiq.transmission.xacro" />
     <xacro:robotiq_transmission prefix="${name}_finger" reduction="${reduction}" />
@@ -78,52 +58,22 @@
       <state_interface name="effort" />
     </joint>
-    <joint name="${name}_right_outer_knuckle_joint">
-      <param name="mimic">${name}_finger_joint</param>
-      <param name="multiplier">-1</param>
-      <command_interface name="position"/>
-      <state_interface name="position"/>
-      <state_interface name="velocity"/>
-      <state_interface name="effort"/>
-    </joint>
-    <joint name="${name}_right_inner_knuckle_joint">
-      <param name="mimic">${name}_finger_joint</param>
-      <param name="multiplier">-1</param>
-      <command_interface name="position"/>
-      <state_interface name="position"/>
-      <state_interface name="velocity"/>
-      <state_interface name="effort"/>
-    </joint>
-    <joint name="${name}_right_inner_finger_joint">
-      <param name="mimic">${name}_finger_joint</param>
-      <param name="multiplier">1</param>
-      <command_interface name="position"/>
-      <state_interface name="position"/>
-      <state_interface name="velocity"/>
-      <state_interface name="effort"/>
-    </joint>
-    <joint name="${name}_left_inner_finger_joint">
-      <param name="mimic">${name}_finger_joint</param>
-      <param name="multiplier">1</param>
-      <command_interface name="position"/>
-      <state_interface name="position"/>
-      <state_interface name="velocity"/>
-      <state_interface name="effort"/>
-    </joint>
-    <joint name="${name}_left_inner_knuckle_joint">
-      <param name="mimic">${name}_finger_joint</param>
-      <param name="multiplier">-1</param>
-      <command_interface name="position"/>
-      <state_interface name="position"/>
-      <state_interface name="velocity"/>
-      <state_interface name="effort"/>
-    </joint>
-    <joint name="${name}_left_outer_knuckle_joint">
-      <param name="mimic">${name}_finger_joint</param>
-      <param name="multiplier">1</param>
-      <command_interface name="position"/>
-      <state_interface name="position"/>
-      <state_interface name="velocity"/>
-      <state_interface name="effort"/>
-    </joint>
+    <xacro:ros2_control_mimic_joint mimic_joint_name="${name}_right_outer_knuckle_joint"
+                                    actuated_joint_name="${name}_finger_joint"
+                                    multiplier="1"/>
+    <xacro:ros2_control_mimic_joint mimic_joint_name="${name}_right_inner_knuckle_joint"
+                                    actuated_joint_name="${name}_finger_joint"
+                                    multiplier="1"/>
+    <xacro:ros2_control_mimic_joint mimic_joint_name="${name}_right_inner_finger_joint"
+                                    actuated_joint_name="${name}_finger_joint"
+                                    multiplier="-1"/>
+    <xacro:ros2_control_mimic_joint mimic_joint_name="${name}_left_inner_finger_joint"
+                                    actuated_joint_name="${name}_finger_joint"
+                                    multiplier="-1"/>
+    <xacro:ros2_control_mimic_joint mimic_joint_name="${name}_left_inner_knuckle_joint"
+                                    actuated_joint_name="${name}_finger_joint"
+                                    multiplier="1"/>
+    <xacro:ros2_control_mimic_joint mimic_joint_name="${name}_left_outer_knuckle_joint"
+                                    actuated_joint_name="${name}_finger_joint"
+                                    multiplier="1"/>
     <xacro:include filename="$(find pal_robotiq_description)/urdf/robotiq.transmission.xacro" />
     <xacro:robotiq_transmission prefix="${name}_finger" reduction="${reduction}" />
